File: hardware/audio_amp_r2/audio_amp_r2.kicad_pcb (KiCad board)
At the start: 2 copper layers, 92 x 35 mm, 29 parts, among them J1 PJ-320D, J2 PJ-320D, J3 JST_PH_1x02, J6 KH-BNC50-3511, J7 KH-BNC50-3511, J8 Conn_01x04_Pin, U1 AD8397

Commit message: update input / output gain levels
Parts:
- R12: value 100R -> 10R
- R4: value 22K -> 100k
- moved R12 15.7 mm to (86.0, 140.2), turned to 0 degrees
- moved R4 12.5 mm to (79.5, 140.1), turned to 180 degrees
- moved R7 12.3 mm to (106.6, 130.4), turned to 180 degrees
- moved R9 5.79 mm to (96.8, 133.3), turned to 180 degrees
- moved J8 2.51 mm to (78.6, 144.3)
- moved C6 1.87 mm to (101.1, 133.3)
Routing:
- net Net-(C7-Pad2): track 17.6 -> 0.00 mm
- net Net-(C6-Pad1): track 15.0 -> 2.47 mm, vias 2 -> 0
- net /Mic: track 45.7 -> 52.2 mm
- net Net-(J8-Pin_2): track 25.0 -> 29.2 mm
- net Net-(J8-Pin_3): track 31.8 -> 35.5 mm
- net Net-(J8-Pin_4): track 28.5 -> 31.9 mm
- net Net-(U1B--): track 9.68 -> 12.8 mm
- net /Left: track 71.4 -> 73.6 mm
- net Net-(J8-Pin_1): track 25.8 -> 24.0 mm

Commit message: add power supply to audio test board
Parts:
- added C10: 10uF, Capacitor_Tantalum_SMD:CP_EIA-3216-18_Kemet-A, F.Cu at (55.9, 125.5)
- added C9: 0.1uF, Capacitor_SMD:C_0805_2012Metric, F.Cu at (55.9, 120.8)
- added U2: AMS1117-3.3, Package_TO_SOT_SMD:SOT-223-3_TabPin2, F.Cu at (49.5, 124.0)
- moved C4 13.0 mm to (64.3, 127.9)
- moved J3 12.6 mm to (64.2, 120.5)
Connections:
- C4 pad 1: +3.3V -> Net-(J3-Pin_2)
- J3 pad 2: +3.3V -> Net-(J3-Pin_2)
Routing:
- net GND: track 286.0 -> 335.6 mm, vias 6 -> 8
- net Net-(J3-Pin_2): track 0.00 -> 20.3 mm
- net +3.3V: track 98.9 -> 89.9 mm
- net Net-(C7-Pad2): track 0.00 -> 3.88 mm
- net Net-(J6-In): track 43.6 -> 44.7 mm
- net /Left: track 73.6 -> 74.6 mm
- added copper zone on F.Cu, net +3.3V

Commit message: move audio board to R2 build
Parts:
- moved C6 1.11 mm to (102.2, 133.3)
- moved C7 0.21 mm to (112.1, 130.4)
- moved R6 0.18 mm to (117.5, 130.4)
Routing:
- net /Left: track 74.6 -> 68.7 mm
- net /Mic: track 52.2 -> 49.3 mm
- net GND: track 335.6 -> 333.9 mm
- net Net-(J8-Pin_4): track 31.9 -> 30.3 mm
- net Net-(C6-Pad1): track 2.47 -> 3.59 mm
- net +3.3V: track 89.9 -> 89.2 mm

Commit message: version sent for R2build of audio amp HW
Changed lines of the file:
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@@
     (descr "SOIC, 8 Pin (JEDEC MS-012AA, https://www.analog.com/media/en/package-pcb-resources/package/pkg_pdf/soic_narrow-r/r_8.pdf), generated with kicad-footprint-generator ipc_gullwing_generator.py")
     (tags "SOIC SO")
-    (property "JLCPCB Part #" "C578714")
+    (property "JLCPCB Part #" "C90876")
     (property "Sheetfile" "audio_amp_r2.kicad_sch")
     (property "Sheetname" "")
@@
     (property "Sim.Enable" "0")
     (property "dnp" "")
-    (property "exclude_from_bom" "")
     (property "ki_description" "Generic connector, single row, 01x04, script generated")
     (property "ki_keywords" "connector")
-    (attr through_hole exclude_from_bom)
+    (attr through_hole)
     (fp_text reference "J8" (at 0 -2.33 90) (layer "F.SilkS") hide
         (effects (font (size 1 1) (thickness 0.15)))
@@
   (segment (start 79.348243 126.082174) (end 79.348243 123.52968) (width 0.25) (layer "F.Cu") (net 8))
   (segment (start 79.348243 123.52968) (end 79.322678 123.504115) (width 0.25) (layer "F.Cu") (net 8))
+  (segment (start 81.13279 134.51738) (end 81.20345 134.44672) (width 0.25) (layer "F.Cu") (net 9))
+  (segment (start 76.719456 131.937454) (end 79.299382 134.51738) (width 0.25) (layer "F.Cu") (net 9))
   (segment (start 76.773565 124.39757) (end 76.663862 124.287867) (width 0.25) (layer "F.Cu") (net 9))
   (segment (start 76.773565 126.585927) (end 76.773565 124.39757) (width 0.25) (layer "F.Cu") (net 9))
-  (segment (start 81.13279 134.51738) (end 81.20345 134.44672) (width 0.25) (layer "F.Cu") (net 9))
-  (segment (start 79.131352 134.51738) (end 81.13279 134.51738) (width 0.25) (layer "F.Cu") (net 9))
-  (segment (start 76.719456 131.930484) (end 76.631956 132.017984) (width 0.25) (layer "F.Cu") (net 9))
+  (segment (start 76.719456 128.987867) (end 76.719456 131.937454) (width 0.25) (layer "F.Cu") (net 9))
   (segment (start 76.719456 128.987867) (end 76.719456 126.640036) (width 0.25) (layer "F.Cu") (net 9))
-  (segment (start 76.719456 128.987867) (end 76.719456 131.930484) (width 0.25) (layer "F.Cu") (net 9))
-  (segment (start 76.631956 132.017984) (end 79.131352 134.51738) (width 0.25) (layer "F.Cu") (net 9))
+  (segment (start 79.299382 134.51738) (end 81.13279 134.51738) (width 0.25) (layer "F.Cu") (net 9))
   (segment (start 90.778017 137.321191) (end 87.94729 140.151918) (width 0.25) (layer "F.Cu") (net 10))
   (segment (start 86.897221 140.151918) (end 86.897221 141.524238) (width 0.25) (layer "F.Cu") (net 10))
