File: hardware/blink_v6/blink_v6.kicad_sch (KiCad schematic)
At the start: 78 parts, among them J1 Conn_01x02, J14 Conn_02x16_Odd_Even, J5 Conn_01x04_Pin, J6 Conn_01x04_Pin, J7 Conn_01x06_Pin, J8 Conn_01x06, J9 Conn_01x04_Pin, U1 AMS1117-3.3, U3 M24C02-RMN, U4 STM32F405RGTx, U5 SN74LVC1G14DBV, U6 SN74LVC1G14DBV, X1 GTXO-14V (2.048MHz), Y1 16MHz

Commit message: part placement
Parts:
- removed J9: Conn_01x04_Pin, Connector_PinHeader_2.54mm:PinHeader_1x04_P2.54mm_Vertical, symbol Connector:Conn_01x04_Pin
- added C?: 10uF, Capacitor_SMD:C_0805_2012Metric, symbol Device:C_Small
- added R? (x2): 560R, Resistor_SMD:R_0805_2012Metric, symbol Device:R_Small_US
- J?: footprint Connector_PinHeader_2.54mm:PinHeader_1x04_P2.54mm_Vertical_SMD_Pin1Left -> Connector_PinHeader_2.54mm:PinHeader_1x04_P2.54mm_Vertical; now not fitted; now left out of the parts list
Connections:
- net AUD_IN: now also R?.1
- net AUD_OUT: now also R?.2
- net at J?.2 (Pin_2), R?.1, R?.2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: now also R?.2
- net at C?.2, R?.1: now also C?.2
- new net: C?.1, R?.1
Changed lines of the file:
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@@
   (junction (at 356.87 339.09) (diameter 0) (color 0 0 0 0)
   )
+  (junction (at 168.91 314.96) (diameter 0) (color 0 0 0 0)
+  )
   (junction (at 33.02 81.28) (diameter 0) (color 0 0 0 0)
   )
@@
     (stroke (width 0) (type default))
   )
-  (wire (pts (xy 172.72 314.96) (xy 162.56 314.96))
+  (wire (pts (xy 172.72 314.96) (xy 168.91 314.96))
     (stroke (width 0) (type default))
   )
@@
     (stroke (width 0) (type default))
   )
+  (wire (pts (xy 177.8 304.8) (xy 182.88 304.8))
+    (stroke (width 0) (type default))
+  )
   (wire (pts (xy 232.41 205.74) (xy 232.41 212.09))
     (stroke (width 0) (type default))
@@
     (stroke (width 0) (type default))
   )
+  (wire (pts (xy 168.91 304.8) (xy 168.91 314.96))
+    (stroke (width 0) (type default))
+  )
   (wire (pts (xy 199.39 320.04) (xy 199.39 331.47))
     (stroke (width 0) (type default))
@@
     (stroke (width 0) (type default))
   )
+  (wire (pts (xy 172.72 304.8) (xy 168.91 304.8))
+    (stroke (width 0) (type default))
+  )
   (wire (pts (xy 392.43 318.77) (xy 392.43 323.85))
     (stroke (width 0) (type default))
@@
     (stroke (width 0) (type default))
   )
+  (wire (pts (xy 182.88 276.86) (xy 173.99 276.86))
+    (stroke (width 0) (type default))
+  )
   (wire (pts (xy 191.77 356.87) (xy 191.77 355.6))
     (stroke (width 0) (type default))
@@
     (stroke (width 0) (type default))
   )
+  (wire (pts (xy 168.91 314.96) (xy 162.56 314.96))
+    (stroke (width 0) (type default))
+  )
   (wire (pts (xy 218.44 72.39) (xy 218.44 76.2))
     (stroke (width 0) (type default))
@@
     (stroke (width 0) (type default))
   )
+  (wire (pts (xy 173.99 276.86) (xy 173.99 287.02))
+    (stroke (width 0) (type default))
+  )
   (wire (pts (xy 384.81 351.79) (xy 392.43 351.79))
     (stroke (width 0) (type default))
@@
     (effects (font (size 1.27 1.27)) (justify right bottom))
   )
+  (label "AUD_IN" (at 187.96 276.86 0) (fields_autoplaced)
+    (effects (font (size 1.27 1.27)) (justify left bottom))
+  )
   (label "DB3" (at 133.35 133.35 0) (fields_autoplaced)
     (effects (font (size 1.27 1.27)) (justify left bottom))
@@
     (effects (font (size 1.27 1.27)) (justify left bottom))
   )
+  (label "AUD_OUT" (at 187.96 304.8 0) (fields_autoplaced)
+    (effects (font (size 1.27 1.27)) (justify left bottom))
+  )
   (label "LEDB" (at 309.88 142.24 0) (fields_autoplaced)
     (effects (font (size 1.27 1.27)) (justify left bottom))
@@
     (effects (font (size 1.27 1.27)) (justify left bottom))
   )
-  (label "AUD_OUT" (at 248.92 298.45 0) (fields_autoplaced)
-    (effects (font (size 1.27 1.27)) (justify left bottom))
-  )
-  (label "AUD_IN" (at 248.92 300.99 0) (fields_autoplaced)
-    (effects (font (size 1.27 1.27)) (justify left bottom))
-  )
   (label "LEDM2" (at 331.47 149.86 0) (fields_autoplaced)
     (effects (font (size 1.27 1.27)) (justify left bottom))
@@
     )
   )
+  (symbol (lib_id "Device:R_Small_US") (at 185.42 276.86 270) (unit 1)
+    (in_bom yes) (on_board yes) (dnp no) (fields_autoplaced)
+    (property "Reference" "R?" (at 185.42 270.51 90)
+      (effects (font (size 1.27 1.27)))
+    )
+    (property "Value" "560R" (at 185.42 273.05 90)
+      (effects (font (size 1.27 1.27)))
+    )
+    (property "Footprint" "Resistor_SMD:R_0805_2012Metric" (at 185.42 276.86 0)
+      (effects (font (size 1.27 1.27)) hide)
+    )
+    (property "Datasheet" "~" (at 185.42 276.86 0)
+      (effects (font (size 1.27 1.27)) hide)
+    )
+    (property "JLCPCB Part #" "C28636" (at 185.42 276.86 0)
+      (effects (font (size 1.27 1.27)) hide)
+    )
+    (pin "1")
+    (pin "2")
+    (instances
+      (project "audio_amp_r1"
+        (path "/65a2a7ad-257a-48a0-a706-3da4b4be7c88"
+          (reference "R?") (unit 1)
+        )
+      )
+      (project "blink_v6"
+        (path "/bd4d3b9a-07c1-4a53-9c94-2893f3e869d4"
+          (reference "R1") (unit 1)
+        )
+      )
+    )
+  )
   (symbol (lib_id "power:GND") (at 162.56 101.6 0) (unit 1)
     (in_bom yes) (on_board yes) (dnp no) (fields_autoplaced)
@@
   )
   (symbol (lib_id "Connector:Conn_01x04_Pin") (at 147.32 308.61 0) (unit 1)
-    (in_bom yes) (on_board yes) (dnp no) (fields_autoplaced)
+    (in_bom no) (on_board yes) (dnp yes) (fields_autoplaced)
     (property "Reference" "J?" (at 147.955 300.99 0)
       (effects (font (size 1.27 1.27)))
@@
       (effects (font (size 1.27 1.27)))
     )
-    (property "Footprint" "Connector_PinHeader_2.54mm:PinHeader_1x04_P2.54mm_Vertical_SMD_Pin1Left" (at 147.32 308.61 0)
+    (property "Footprint" "Connector_PinHeader_2.54mm:PinHeader_1x04_P2.54mm_Vertical" (at 147.32 308.61 0)
       (effects (font (size 1.27 1.27)) hide)
     )
@@
     )
   )
-  (symbol (lib_id "power:GND") (at 248.92 303.53 0) (unit 1)
-    (in_bom yes) (on_board yes) (dnp no)
-    (property "Reference" "#PWR023" (at 248.92 309.88 0)
-      (effects (font (size 1.27 1.27)) hide)
-    )
-    (property "Value" "GND" (at 248.92 307.34 0)
-      (effects (font (size 1.27 1.27)))
-    )
-    (property "Footprint" "" (at 248.92 303.53 0)
-      (effects (font (size 1.27 1.27)) hide)
-    )
-    (property "Datasheet" "" (at 248.92 303.53 0)
-      (effects (font (size 1.27 1.27)) hide)
-    )
-    (pin "1")
-    (instances
-      (project "blink_v6"
-        (path "/bd4d3b9a-07c1-4a53-9c94-2893f3e869d4"
-          (reference "#PWR023") (unit 1)
-        )
-      )
-    )
-  )
   (symbol (lib_id "Device:R_Small_US") (at 341.63 322.58 0) (unit 1)
     (in_bom yes) (on_board yes) (dnp no) (fields_autoplaced)
@@
     )
   )
-  (symbol (lib_id "Connector:Conn_01x04_Pin") (at 243.84 298.45 0) (unit 1)
-    (in_bom no) (on_board yes) (dnp yes) (fields_autoplaced)
-    (property "Reference" "J9" (at 242.57 300.99 0)
-      (effects (font (size 1.27 1.27)) (justify right))
-    )
-    (property "Value" "Conn_01x04_Pin" (at 242.57 298.45 0)
-      (effects (font (size 1.27 1.27)) (justify right) hide)
-    )
-    (property "Footprint" "Connector_PinHeader_2.54mm:PinHeader_1x04_P2.54mm_Vertical" (at 243.84 298.45 0)
-      (effects (font (size 1.27 1.27)) hide)
-    )
-    (property "Datasheet" "~" (at 243.84 298.45 0)
-      (effects (font (size 1.27 1.27)) hide)
-    )
-    (pin "1")
-    (pin "2")
-    (pin "3")
-    (pin "4")
-    (instances
-      (project "blink_v6"
-        (path "/bd4d3b9a-07c1-4a53-9c94-2893f3e869d4"
-          (reference "J9") (unit 1)
-        )
-      )
-    )
-  )
-  (symbol (lib_id "power:+3.3VA") (at 248.92 295.91 0) (unit 1)
-    (in_bom yes) (on_board yes) (dnp no) (fields_autoplaced)
-    (property "Reference" "#PWR022" (at 248.92 299.72 0)
-      (effects (font (size 1.27 1.27)) hide)
-    )
-    (property "Value" "+3.3VA" (at 248.92 290.83 0)
-      (effects (font (size 1.27 1.27)))
-    )
-    (property "Footprint" "" (at 248.92 295.91 0)
-      (effects (font (size 1.27 1.27)) hide)
-    )
-    (property "Datasheet" "" (at 248.92 295.91 0)
-      (effects (font (size 1.27 1.27)) hide)
-    )
-    (pin "1")
-    (instances
-      (project "blink_v6"
-        (path "/bd4d3b9a-07c1-4a53-9c94-2893f3e869d4"
-          (reference "#PWR022") (unit 1)
-        )
-      )
-    )
-  )
   (symbol (lib_id "Device:C_Polarized_Small_US") (at 90.17 257.81 0) (unit 1)
     (in_bom yes) (on_board yes) (dnp no) (fields_autoplaced)
@@
     )
   )
+  (symbol (lib_id "Device:C_Small") (at 175.26 304.8 270) (unit 1)
+    (in_bom yes) (on_board yes) (dnp no) (fields_autoplaced)
+    (property "Reference" "C?" (at 175.2536 298.45 90)
+      (effects (font (size 1.27 1.27)))
+    )
+    (property "Value" "10uF" (at 175.2536 300.99 90)
+      (effects (font (size 1.27 1.27)))
+    )
+    (property "Footprint" "Capacitor_SMD:C_0805_2012Metric" (at 175.26 304.8 0)
+      (effects (font (size 1.27 1.27)) hide)
+    )
+    (property "Datasheet" "~" (at 175.26 304.8 0)
+      (effects (font (size 1.27 1.27)) hide)
+    )
+    (property "JLCPCB Part #" "C15850" (at 175.26 304.8 0)
+      (effects (font (size 1.27 1.27)) hide)
+    )
+    (pin "1")
+    (pin "2")
+    (instances
+      (project "audio_amp_r1"
+        (path "/65a2a7ad-257a-48a0-a706-3da4b4be7c88"
+          (reference "C?") (unit 1)
+        )
+      )
+      (project "blink_v6"
+        (path "/bd4d3b9a-07c1-4a53-9c94-2893f3e869d4"
+          (reference "C26") (unit 1)
+        )
+      )
+    )
+  )
   (symbol (lib_id "Device:C_Small") (at 175.26 314.96 270) (unit 1)
     (in_bom yes) (on_board yes) (dnp no) (fields_autoplaced)
@@
         )
       )
+    )
+  )
+  (symbol (lib_id "Device:R_Small_US") (at 185.42 304.8 90) (unit 1)
+    (in_bom yes) (on_board yes) (dnp no) (fields_autoplaced)
+    (property "Reference" "R?" (at 185.42 298.45 90)
+      (effects (font (size 1.27 1.27)))
+    )
+    (property "Value" "560R" (at 185.42 300.99 90)
+      (effects (font (size 1.27 1.27)))
+    )
+    (property "Footprint" "Resistor_SMD:R_0805_2012Metric" (at 185.42 304.8 0)
+      (effects (font (size 1.27 1.27)) hide)
+    )
+    (property "Datasheet" "~" (at 185.42 304.8 0)
+      (effects (font (size 1.27 1.27)) hide)
+    )
+    (property "JLCPCB Part #" "C28636" (at 185.42 304.8 0)
+      (effects (font (size 1.27 1.27)) hide)
+    )
+    (pin "1")
+    (pin "2")
+    (instances
+      (project "audio_amp_r1"
+        (path "/65a2a7ad-257a-48a0-a706-3da4b4be7c88"
+          (reference "R?") (unit 1)
+        )
+      )
+      (project "blink_v6"
+        (path "/bd4d3b9a-07c1-4a53-9c94-2893f3e869d4"
+          (reference "R19") (unit 1)
+        )
+      )

Commit message: signal routing done
Connections:
- net AUX_CLK: now also J14.29 (Pin_29)
- net AUX_GPS_PPS: now also J14.31 (Pin_31)
- net AUX_SYNC_MON: now also J14.32 (Pin_32)
- net BOOT1: now also J14.21 (Pin_21)
- net COL1: now also J14.27 (Pin_27); no longer J14.7 (Pin_7)
- net COL2: now also J14.28 (Pin_28); no longer J14.10 (Pin_10)
- net COL3: now also J14.26 (Pin_26); no longer J14.6 (Pin_6)
- net COL4: now also J14.24 (Pin_24); no longer J14.8 (Pin_8)
- net COL5: now also J14.23 (Pin_23); no longer J14.5 (Pin_5)
- net LEDA: now also J14.15 (Pin_15); no longer J14.27 (Pin_27)
- net LEDB: now also J14.6 (Pin_6); no longer J14.19 (Pin_19)
- net LEDC: now also J14.5 (Pin_5); no longer J14.20 (Pin_20)
- net LEDD: now also J14.8 (Pin_8); no longer J14.17 (Pin_17)
- net LEDE: now also J14.7 (Pin_7); no longer J14.18 (Pin_18)
- net LEDF: now also J14.14 (Pin_14); no longer J14.11 (Pin_11)
- net LEDG: now also J14.13 (Pin_13); no longer J14.12 (Pin_12)
- net LEDH: now also J14.16 (Pin_16); no longer J14.9 (Pin_9)
- net LEDM1: now also J14.17 (Pin_17); no longer J14.23 (Pin_23)
- net LEDM2: now also J14.30 (Pin_30); no longer J14.26 (Pin_26)
- net LEDM3: now also J14.18 (Pin_18); no longer J14.25 (Pin_25)
- net ROW1: now also J14.10 (Pin_10); no longer J14.15 (Pin_15)
- net ROW2: now also J14.9 (Pin_9); no longer J14.16 (Pin_16)
- net ROW3: now also J14.12 (Pin_12); no longer J14.13 (Pin_13)
- net ROW4: now also J14.11 (Pin_11); no longer J14.14 (Pin_14)
- net ROW5: now also J14.25 (Pin_25); no longer J14.28 (Pin_28)
- net ROW6: now also J14.20 (Pin_20); no longer J14.22 (Pin_22)
- net ROW7: now also J14.19 (Pin_19); no longer J14.21 (Pin_21)
- net ROW8: now also J14.22 (Pin_22); no longer J14.24 (Pin_24)

Commit message: change mic in out gains
Parts:
- R?: value 22K -> 100K; JLCPCB Part # C17560 -> C149504
- R?: value 100R -> 10R; JLCPCB Part # C17408 -> C17415
Changed lines of the file:
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@@
       (effects (font (size 1.27 1.27)))
     )
-    (property "Value" "22K" (at 163.83 292.1 90)
+    (property "Value" "100K" (at 163.83 292.1 90)
       (effects (font (size 1.27 1.27)))
     )
@@
       (effects (font (size 1.27 1.27)) hide)
     )
-    (property "JLCPCB Part #" "C17560" (at 163.83 295.91 0)
+    (property "JLCPCB Part #" "C149504" (at 163.83 295.91 0)
       (effects (font (size 1.27 1.27)) hide)
     )
@@
       (effects (font (size 1.27 1.27)) (justify left))
     )
-    (property "Value" "100R" (at 165.1 346.71 0)
+    (property "Value" "10R" (at 165.1 346.71 0)
       (effects (font (size 1.27 1.27)) (justify left))
     )
@@
       (effects (font (size 1.27 1.27)) hide)
     )
-    (property "JLCPCB Part #" "C17408" (at 162.56 345.44 0)
-      (effects (font (size 1.27 1.27)) hide)
-    )
+    (property "JLCPCB Part #" "C17415" (at 162.56 345.44 0)
+      (effects (font (size 1.27 1.27)) hide)
+    )

Commit message: reduce schematic paper size
Other:
- title: Blinky V4 -> Blinky V6
- moved on the sheet: C1, C10, C11, C12, C14, C15, C16, C18, C19, C2, C20, C21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
