File: hardware/disp_v6/disp_v6.kicad_pcb (KiCad board)
At the start: 2 copper layers, 82 x 52 mm, 109 parts, among them J1 Conn_02x16_Odd_Even, Q1 2N7002, Q10 2N7002, Q11 2N7002, Q2 2N7002, Q3 2N7002, Q4 2N7002, Q5 2N7002, Q6 2N7002, Q7 2N7002, Q8 2N7002, Q9 2N7002

Commit message: dreive new ros off of boot0 boot1
Connections:
- net /AUX_CLK renamed /BOOT0
- net /AUX_SYNC_MON renamed /GPS_PPS
- R1 pad 2: /AUX_GPS_PPS -> /BOOT1
Routing:
- net /AUX_GPS_PPS: track 15.7 -> 0.00 mm, vias 1 -> 0
- net /BOOT1: track 0.00 -> 12.1 mm
Changed lines of the file:
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@@
   (net 56 "Net-(Q10-D)")
   (net 57 "/BOOT1")
-  (net 58 "/AUX_CLK")
+  (net 58 "/BOOT0")
   (net 59 "/AUX_GPS_PPS")
-  (net 60 "/AUX_SYNC_MON")
+  (net 60 "/GPS_PPS")
   (net 61 "Net-(Q11-D)")
   (net 62 "/R9")
@@
       (net 63 "/R0") (pintype "passive"))
     (pad "2" smd roundrect (at 0.825 0 90) (size 0.8 0.95) (layers "F.Cu" "F.Paste" "F.Mask") (roundrect_rratio 0.25)
-      (net 58 "/AUX_CLK") (pintype "passive"))
+      (net 58 "/BOOT0") (pintype "passive"))
     (model "${KICAD6_3DMODEL_DIR}/Resistor_SMD.3dshapes/R_0603_1608Metric.wrl"
       (offset (xyz 0 0 0))
@@
       (net 62 "/R9") (pintype "passive"))
     (pad "2" smd roundrect (at 0.825 0 90) (size 0.8 0.95) (layers "F.Cu" "F.Paste" "F.Mask") (roundrect_rratio 0.25)
-      (net 59 "/AUX_GPS_PPS") (pintype "passive"))
+      (net 57 "/BOOT1") (pintype "passive"))
     (model "${KICAD6_3DMODEL_DIR}/Resistor_SMD.3dshapes/R_0603_1608Metric.wrl"
       (offset (xyz 0 0 0))
@@
       (net 8 "/COL2") (pinfunction "Pin_28") (pintype "passive"))
     (pad "29" thru_hole oval locked (at 0 -35.56 90) (size 1.7 1.7) (drill 1) (layers "*.Cu" "*.Mask")
-      (net 58 "/AUX_CLK") (pinfunction "Pin_29") (pintype "passive"))
+      (net 58 "/BOOT0") (pinfunction "Pin_29") (pintype "passive"))
     (pad "30" thru_hole oval locked (at 2.709399 -35.804651 90) (size 1.7 1.7) (drill 1) (layers "*.Cu" "*.Mask")
       (net 4 "/LEDM2") (pinfunction "Pin_30") (pintype "passive"))
@@
       (net 59 "/AUX_GPS_PPS") (pinfunction "Pin_31") (pintype "passive"))
     (pad "32" thru_hole oval locked (at 2.54 -38.1 90) (size 1.7 1.7) (drill 1) (layers "*.Cu" "*.Mask")
-      (net 60 "/AUX_SYNC_MON") (pinfunction "Pin_32") (pintype "passive"))
+      (net 60 "/GPS_PPS") (pinfunction "Pin_32") (pintype "passive"))
     (model "${KICAD6_3DMODEL_DIR}/Connector_PinHeader_2.54mm.3dshapes/PinHeader_2x16_P2.54mm_Vertical.wrl"
       (offset (xyz 0 0 0))
@@
   (segment (start 202.996474 90.446599) (end 202.996474 92.014148) (width 0.15) (layer "F.Cu") (net 50))
   (segment (start 202.996474 107.981378) (end 202.977852 108) (width 0.15) (layer "F.Cu") (net 50))
-  (segment (start 205.445306 80.257607) (end 205.445306 85.640366) (width 0.15) (layer "F.Cu") (net 51))
-  (segment (start 205.561011 80.141902) (end 205.445306 80.257607) (width 0.15) (layer "F.Cu") (net 51))
-  (via (at 205.561011 80.141902) (size 0.8) (drill 0.4) (layers "F.Cu" "B.Cu") (net 51))
+  (segment (start 205.561011 81.17485) (end 205.445306 81.290555) (width 0.15) (layer "F.Cu") (net 51))
+  (segment (start 205.445306 81.290555) (end 205.445306 85.640366) (width 0.15) (layer "F.Cu") (net 51))
+  (via (at 205.561011 81.17485) (size 0.8) (drill 0.4) (layers "F.Cu" "B.Cu") (net 51))
+  (segment (start 205.561011 81.17485) (end 205.561011 80.141902) (width 0.15) (layer "B.Cu") (net 51))
   (segment (start 205.561011 80.141902) (end 202.52 77.100891) (width 0.15) (layer "B.Cu") (net 51))
   (segment (start 202.52 77.100891) (end 202.52 76) (width 0.15) (layer "B.Cu") (net 51))
@@
   (segment (start 238.667666 92.057596) (end 238.702173 92.092103) (width 0.15) (layer "F.Cu") (net 56))
   (segment (start 236.621336 92.057596) (end 238.667666 92.057596) (width 0.15) (layer "F.Cu") (net 56))
-  (segment (start 199.36042 80.97485) (end 203.88492 80.97485) (width 0.15) (layer "F.Cu") (net 58))
-  (segment (start 199.28492 80.89935) (end 199.36042 80.97485) (width 0.15) (layer "F.Cu") (net 58))
+  (segment (start 204.88492 80.07485) (end 203.48492 81.47485) (width 0.15) (layer "F.Cu") (net 57))
+  (segment (start 207.6 78.65977) (end 206.18492 80.07485) (width 0.15) (layer "F.Cu") (net 57))
+  (segment (start 206.18492 80.07485) (end 204.88492 80.07485) (width 0.15) (layer "F.Cu") (net 57))
+  (segment (start 207.6 76) (end 207.6 78.65977) (width 0.15) (layer "F.Cu") (net 57))
+  (segment (start 203.48492 81.47485) (end 203.48492 85.64985) (width 0.15) (layer "F.Cu") (net 57))
+  (segment (start 202.48492 80.97485) (end 199.36042 80.97485) (width 0.15) (layer "F.Cu") (net 58))
+  (segment (start 199.36042 80.97485) (end 199.28492 80.89935) (width 0.15) (layer "F.Cu") (net 58))
   (segment (start 218.98492 82.67485) (end 218.98492 85.47485) (width 0.15) (layer "F.Cu") (net 58))
   (segment (start 218.98492 85.47485) (end 219.08492 85.57485) (width 0.15) (layer "F.Cu") (net 58))
-  (segment (start 203.88492 80.97485) (end 204.58492 81.67485) (width 0.15) (layer "F.Cu") (net 58))
   (via (at 218.98492 82.67485) (size 0.8) (drill 0.4) (layers "F.Cu" "B.Cu") (net 58))
-  (via (at 204.58492 81.67485) (size 0.8) (drill 0.4) (layers "F.Cu" "B.Cu") (net 58))
+  (via (at 202.48492 80.97485) (size 0.8) (drill 0.4) (layers "F.Cu" "B.Cu") (net 58))
   (via (at 199.28492 80.89935) (size 0.8) (drill 0.4) (layers "F.Cu" "B.Cu") (net 58))
-  (segment (start 205.58492 82.67485) (end 218.98492 82.67485) (width 0.15) (layer "B.Cu") (net 58))
   (segment (start 199.28492 80.89935) (end 197.44 79.05443) (width 0.15) (layer "B.Cu") (net 58))
-  (segment (start 204.58492 81.67485) (end 205.58492 82.67485) (width 0.15) (layer "B.Cu") (net 58))
   (segment (start 197.44 79.05443) (end 197.44 76) (width 0.15) (layer "B.Cu") (net 58))
-  (segment (start 198.18492 81.37485) (end 198.38442 81.57435) (width 0.15) (layer "F.Cu") (net 59))
-  (segment (start 202.38442 81.57435) (end 203.48492 82.67485) (width 0.15) (layer "F.Cu") (net 59))
-  (segment (start 198.38442 81.57435) (end 202.38442 81.57435) (width 0.15) (layer "F.Cu") (net 59))
-  (segment (start 203.48492 82.67485) (end 203.48492 85.64985) (width 0.15) (layer "F.Cu") (net 59))
-  (via (at 198.18492 81.37485) (size 0.8) (drill 0.4) (layers "F.Cu" "B.Cu") (net 59))
-  (segment (start 197.88492 81.37485) (end 194.9 78.38993) (width 0.15) (layer "B.Cu") (net 59))
-  (segment (start 198.18492 81.37485) (end 197.88492 81.37485) (width 0.15) (layer "B.Cu") (net 59))
-  (segment (start 194.9 78.38993) (end 194.9 76) (width 0.15) (layer "B.Cu") (net 59))
+  (segment (start 204.18492 82.67485) (end 218.98492 82.67485) (width 0.15) (layer "B.Cu") (net 58))
+  (segment (start 202.48492 80.97485) (end 204.18492 82.67485) (width 0.15) (layer "B.Cu") (net 58))
   (segment (start 236.621336 99.557596) (end 238.679551 99.557596) (width 0.15) (layer "F.Cu") (net 61))
   (segment (start 238.679551 99.557596) (end 238.693221 99.543926) (width 0.15) (layer "F.Cu") (net 61))

Commit message: update rotations
Parts:
- D10, D11, D4, D5, D6, D7, D8, D9: value LED-RED -> LED-R
