File: hardware/clock_v6/clock_v6.kicad_sch (KiCad schematic)
At the start: 151 parts, among them J1 RJ45, J12 Conn_01x06, J2 Conn_01x06_Pin, J4 Conn_01x04_Pin, J5 Conn_01x06_Pin, J6 Conn_01x04_Pin, J7 Conn_01x04_Pin, J8 Conn_01x02, Q10 2N7002, Q9 2N7002, U1 ADA4807-1, U10 STM32F405RGTx, U11 AMS1117-3.3, U12 BA50DD0WHFP-TR, U13 M24C02-RMN, U2 SN74LVC1G14DBV, U3 SN74LVC1G14DBV, U4 ADA4807-1, U5 ADA4807-1, U6 TLV3603DCKR, U7 SN74LVC1G14DBV, U8 TLV3603DCKR, U9 L78L05_SOT89, Y1 AOCJY4A-10.000MHZ-SW, Y2 16MHz

Commit message: ready to go to prod
Parts:
- ANT1, ANT2, ANT3, ANT4, ANT5: JLCPCB Part # (none) -> C88374; JLCPCB Position Offset (none) -> 0,-0.75; JLCPCB Rotation Offset (none) -> 180; LCSC C88374 -> (none)
- C1, C10, C11, C17, C18, C2, C25, C26, C30, C31, C32, C33, C36, C38, C39, C45, C46, C47, C48, C49, C9: JLCPCB Part # (none) -> C307331; LCSC C307331 -> (none)
- C12, C14, C19, C23, C5, C7: JLCPCB Part # (none) -> C1594; LCSC C1594 -> (none)
- C13, C20, C8: JLCPCB Part # (none) -> C1664; LCSC C1664 -> (none)
- C15, C22, C6: JLCPCB Part # (none) -> C1603; LCSC C1603 -> (none)
- C16, C21, C3: JLCPCB Part # (none) -> C1588; LCSC C1588 -> (none)
- C24, C27, C37: JLCPCB Part # (none) -> C14663; LCSC C14663 -> (none)
- C28, C29: JLCPCB Part # (none) -> C1663; LCSC C1663 -> (none)
- C34, C41, C43: JLCPCB Part # (none) -> C7171; LCSC C7171 -> (none)
- C35, C40: JLCPCB Part # (none) -> C23630; LCSC C23630 -> (none)
- C4: JLCPCB Part # (none) -> C14857; LCSC C14857 -> (none)
- C42, C44: JLCPCB Part # (none) -> C128342; LCSC C128342 -> (none)
- D1: JLCPCB Part # (none) -> C94869; LCSC C94869 -> (none)
- D2: JLCPCB Part # (none) -> C125093; LCSC C125093 -> (none)
- D3: JLCPCB Part # (none) -> C72038; LCSC C72038 -> (none)
- FB1: JLCPCB Part # (none) -> C127301; LCSC C127301 -> (none)
- J1: JLCPCB Part # (none) -> C464586; LCSC C464586 -> (none)
- J12: JLCPCB Part # (none) -> C265405; JLCPCB Rotation Offset (none) -> 180; LCSC C265405 -> (none)
- J8: JLCPCB Part # (none) -> C295747; LCSC C295747 -> (none)
- L1, L2, L3, L4, L5, L6: JLCPCB Part # (none) -> C1042; LCSC C1042 -> (none)
- Q10, Q9: JLCPCB Part # (none) -> C8545; JLCPCB Rotation Offset (none) -> 180; LCSC C8545 -> (none)
- R1, R15, R16, R29, R30, R31: JLCPCB Part # (none) -> C22775; LCSC C22775 -> (none)
- R10, R2, R6: JLCPCB Part # (none) -> C23193; LCSC C23193 -> (none)
- R11, R3, R7: JLCPCB Part # (none) -> C23185; LCSC C23185 -> (none)
- R12, R13: JLCPCB Part # (none) -> C4310; LCSC C4310 -> (none)
- R14: JLCPCB Part # (none) -> C17630; LCSC C17630 -> (none)
- R17: JLCPCB Part # (none) -> C17544; LCSC C17544 -> (none)
- R18, R21: JLCPCB Part # (none) -> C22795; LCSC C22795 -> (none)
- R19, R20, R22, R24, R5, R54, R60, R61, R62, R63, R64: JLCPCB Part # (none) -> C21190; LCSC C21190 -> (none)
- R23: JLCPCB Part # (none) -> C17560; LCSC C17560 -> (none)
- R25: JLCPCB Part # (none) -> C22966; LCSC C22966 -> (none)
- R26: JLCPCB Part # (none) -> C23345; LCSC C23345 -> (none)
- R27, R28, R32, R34, R36: JLCPCB Part # (none) -> C23162; LCSC C23162 -> (none)
- R33, R35: JLCPCB Part # (none) -> C4190; LCSC C4190 -> (none)
- R4: JLCPCB Part # (none) -> C17540; LCSC C17540 -> (none)
- R58, R59: JLCPCB Part # (none) -> C22843; LCSC C22843 -> (none)
- R8: JLCPCB Part # (none) -> C17590; LCSC C17590 -> (none)
- R9: JLCPCB Part # (none) -> C17606; LCSC C17606 -> (none)
- U1, U4, U5: JLCPCB Part # (none) -> C2058411; JLCPCB Rotation Offset (none) -> 270; LCSC C2058411 -> (none)
- U10: JLCPCB Part # (none) -> C15742; JLCPCB Rotation Offset (none) -> 270; LCSC C15742 -> (none)
- U11: JLCPCB Part # (none) -> C6186; JLCPCB Rotation Offset (none) -> 180; LCSC C6186 -> (none)
- U12: JLCPCB Part # (none) -> C509718; JLCPCB Position Offset (none) -> -1.5,0; LCSC C509718 -> (none)
- U13: JLCPCB Part # (none) -> C83836; JLCPCB Rotation Offset (none) -> 270; LCSC C83836 -> (none)
- U2, U3, U7: JLCPCB Part # (none) -> C133145; JLCPCB Rotation Offset (none) -> 180; LCSC C133145 -> (none)
- U6, U8: JLCPCB Part # (none) -> C5213955; LCSC C5213955 -> (none)
- U9: JLCPCB Part # (none) -> C71136; JLCPCB Position Offset (none) -> 0.5,0; JLCPCB Rotation Offset (none) -> 180; LCSC C71136 -> (none)
- Y1: JLCPCB Part # (none) -> C1670487; LCSC C1670487 -> (none)
- Y2: JLCPCB Part # (none) -> C13738; LCSC C13738 -> (none)
