File: hardware/disp_v7/disp_v7.kicad_pcb (KiCad board)
At the start: 2 copper layers, 82 x 52 mm, 109 parts, among them J1 Conn_02x16_Odd_Even, Q1 2N7002, Q10 2N7002, Q11 2N7002, Q2 2N7002, Q3 2N7002, Q4 2N7002, Q5 2N7002, Q6 2N7002, Q7 2N7002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

Commit message: update version on disp to v7
Other:
- board text added: "Disp Rev 7.0 Cullen Jennings"
- board text removed: "Disp Rev6.0 Cullen Jennings"
Changed lines of the file:
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@@
   (paper "A4")
   (title_block
-    (title "Blinky V4")
+    (title "Disp")
     (date "2023-07-04")
+    (rev "V7")
     (company "Cullen Jennings")
   )
@@
   (gr_line (start 169 68) (end 169 120)
     (stroke (width 0.1) (type default)) (layer "Edge.Cuts"))
-  (gr_text "Disp Rev6.0	\nCullen Jennings" (at 248.479931 87.842516 90) (layer "F.SilkS")
+  (gr_text "Disp Rev 7.0	\nCullen Jennings" (at 248.479931 87.842516 90) (layer "F.SilkS")
     (effects (font (size 1 1) (thickness 0.15)) (justify left bottom))
   )

Commit message: add switches
Connections:
- net /BOOT0 renamed /ROW10
- net /BOOT1 renamed /ROW9
- J1 pad 31: /AUX_GPS_PPS -> unconnected-(J1-Pin_31-Pad31)
- J1 pad 32: /GPS_PPS -> unconnected-(J1-Pin_32-Pad32)

Commit message: fix up flip connector warning
Parts:
- C32, C36, C38: value 100nF -> 100n
- J1: value Conn_02x16_Odd_Even -> Conn_02x16_Odd_Even_FLIP; footprint Connector_PinHeader_2.54mm:PinHeader_2x16_P2.54mm_Vertical -> blinky_footprints:PinSocket_2x16_P2.54mm_Vertical_FLIP; moved to F.Cu
- turned J1 to -90 degrees
