File: hardware/disp_v8/disp_v8.kicad_pcb (KiCad board)
At the start: 2 copper layers, 82 x 52 mm, 119 parts, among them J1 Conn_02x16_Odd_Even_FLIP, J2 Conn_01x01_Pin, J3 Conn_01x01_Pin, Q1 2N7002, Q10 2N7002, Q11 2N7002, Q12 2N7002, Q13 2N7002, Q2 2N7002, Q3 2N7002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

Commit message: clean up display v8
Parts:
- moved J3 7.12 mm to (194.9, 118.0)
- moved J2 7.11 mm to (233.0, 118.0)
- moved C38 0.97 mm to (233.0, 111.5)
- moved C32 0.33 mm to (236.7, 77.3)
Connections:
- net /LA renamed /L4
- net /LB renamed /L1
- net /LC renamed /L5
- net /LD renamed /L2
- net /LE renamed /L6
- net /LEDG renamed /LED7
- net /LEDH renamed /LED8
- net /LEDM1 renamed /LEDMG
- net /LEDM3 renamed /LEDMY
- net /LF renamed /L3
- net /LG renamed /L7
- net /LH renamed /L8
- net /LI renamed /L9
- net /LJ renamed /L10
- net /R0 renamed /C1
- net /R1 renamed /C5
- net /R2 renamed /C6
- net /R3 renamed /C7
- net /R4 renamed /C8
- net /R5 renamed /C9
- net /R6 renamed /C4
- net /R7 renamed /C3
- net /R8 renamed /C2
- net /R9 renamed /C10
- J1 pad 23: /LEDI -> /LED9
- J1 pad 24: /LEDJ -> /LED10
- J1 pad 27: /NROW2 -> /LED1
- J1 pad 28: /NROW1 -> /LED2
- J1 pad 29: /NCOL1 -> /LED3
- J1 pad 30: /LEDM2 -> /LED4
- J1 pad 31: /LEDJ -> /LED5
- J1 pad 32: /LEDI -> /LED6
- J1 pad 6: /LEDM2 -> /LEDMR
- Q1 pad 1: /LEDA -> /LED4
- Q11 pad 1: /LEDM2 -> /LEDMR
- Q12 pad 1: /LEDI -> /LED9
- Q13 pad 1: /LEDJ -> /LED10
- Q3 pad 1: /LEDF -> /LED3
- Q5 pad 1: /LEDD -> /LED2
- Q6 pad 1: /LEDE -> /LED6
- Q7 pad 1: /LEDB -> /LED1
- Q8 pad 1: /LEDC -> /LED5
- R3 pad 2: /LEDI -> /LED9
- R33 pad 2: /LEDA -> /LED4
- R37 pad 2: /LEDF -> /LED3
- R41 pad 2: /LEDD -> /LED2
- R43 pad 2: /LEDE -> /LED6
- R45 pad 2: /LEDB -> /LED1
- R47 pad 2: /LEDC -> /LED5
- R5 pad 2: /LEDJ -> /LED10
Routing:
- net GND: track 370.9 -> 593.0 mm, vias 8 -> 0
- net /LED1: track 0.00 -> 81.2 mm
- net /LEDB: track 75.6 -> 0.00 mm
- net /LED2: track 0.00 -> 71.4 mm
- net /LEDD: track 68.8 -> 0.00 mm
- net /LED3: track 0.00 -> 68.2 mm
- net /LEDF: track 62.7 -> 0.00 mm
- net /LED4: track 0.00 -> 58.3 mm
- net /LEDA: track 56.0 -> 0.00 mm
- net /LED5: track 0.00 -> 54.1 mm
- net /LEDC: track 48.2 -> 0.00 mm
- net /LED6: track 0.00 -> 41.7 mm
- net /LEDMR: track 0.00 -> 41.1 mm
- net /LEDE: track 40.4 -> 0.00 mm
- net /LED9: track 0.00 -> 40.0 mm
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- added copper zone on F.Cu, net GND

Commit message: order v8 of blink and disp
Parts:
- removed H1, H2, H4, H5: M2, MountingHole:MountingHole_2.2mm_M2
Changed lines of the file:
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@@
     )
   )
-  (footprint "MountingHole:MountingHole_2.2mm_M2" (layer "F.Cu")
-    (at 247.139934 116.451579 90)
-    (descr "Mounting Hole 2.2mm, no annular, M2")
-    (tags "mounting hole 2.2mm no annular m2")
-    (property "Sheetfile" "disp_v8.kicad_sch")
-    (property "Sheetname" "")
-    (property "dnp" "")
-    (property "exclude_from_bom" "")
-    (property "ki_description" "Mounting Hole without connection")
-    (property "ki_keywords" "mounting hole")
-    (attr exclude_from_pos_files exclude_from_bom)
-    (fp_text reference "H4" (at 0 -3.2 90) (layer "F.SilkS") hide
-        (effects (font (size 1 1) (thickness 0.15)))
-    )
-    (fp_text value "M2" (at 0 3.2 90) (layer "F.Fab") hide
-        (effects (font (size 1 1) (thickness 0.15)))
-    )
-    (fp_text user "${REFERENCE}" (at 0 0 90) (layer "F.Fab")
-        (effects (font (size 1 1) (thickness 0.15)))
-    )
-    (fp_circle (center 0 0) (end 2.2 0)
-      (stroke (width 0.15) (type solid)) (fill none) (layer "Cmts.User"))
-    (fp_circle (center 0 0) (end 2.45 0)
-      (stroke (width 0.05) (type solid)) (fill none) (layer "F.CrtYd"))
-    (pad "" np_thru_hole circle (at 0 0 90) (size 2.2 2.2) (drill 2.2) (layers "*.Cu" "*.Mask"))
-  )
   (footprint "LED_SMD:LED_0603_1608Metric" locked (layer "F.Cu")
     (at 205 108)
@@
     )
   )
-  (footprint "MountingHole:MountingHole_2.2mm_M2" (layer "F.Cu")
-    (at 172.774875 71.645227 90)
-    (descr "Mounting Hole 2.2mm, no annular, M2")
-    (tags "mounting hole 2.2mm no annular m2")
-    (property "Sheetfile" "disp_v8.kicad_sch")
-    (property "Sheetname" "")
-    (property "dnp" "")
-    (property "exclude_from_bom" "")
-    (property "ki_description" "Mounting Hole without connection")
-    (property "ki_keywords" "mounting hole")
-    (attr exclude_from_pos_files exclude_from_bom)
-    (fp_text reference "H1" (at 0 -3.2 90) (layer "F.SilkS") hide
-        (effects (font (size 1 1) (thickness 0.15)))
-    )
-    (fp_text value "M2" (at 0 3.2 90) (layer "F.Fab") hide
-        (effects (font (size 1 1) (thickness 0.15)))
-    )
-    (fp_text user "${REFERENCE}" (at 0 0 90) (layer "F.Fab")
-        (effects (font (size 1 1) (thickness 0.15)))
-    )
-    (fp_circle (center 0 0) (end 2.2 0)
-      (stroke (width 0.15) (type solid)) (fill none) (layer "Cmts.User"))
-    (fp_circle (center 0 0) (end 2.45 0)
-      (stroke (width 0.05) (type solid)) (fill none) (layer "F.CrtYd"))
-    (pad "" np_thru_hole circle (at 0 0 90) (size 2.2 2.2) (drill 2.2) (layers "*.Cu" "*.Mask"))
-  )
   (footprint "LED_SMD:LED_0603_1608Metric" (layer "F.Cu")
     (at 229.133334 111.7875 90)
@@
     )
   )
-  (footprint "MountingHole:MountingHole_2.2mm_M2" (layer "F.Cu")
-    (at 172.507561 116.588394)
-    (descr "Mounting Hole 2.2mm, no annular, M2")
-    (tags "mounting hole 2.2mm no annular m2")
-    (property "Sheetfile" "disp_v8.kicad_sch")
-    (property "Sheetname" "")
-    (property "dnp" "")
-    (property "exclude_from_bom" "")
-    (property "ki_description" "Mounting Hole without connection")
-    (property "ki_keywords" "mounting hole")
-    (attr exclude_from_pos_files exclude_from_bom)
-    (fp_text reference "H5" (at 0 -3.2) (layer "F.SilkS") hide
-        (effects (font (size 1 1) (thickness 0.15)))
-    )
-    (fp_text value "M2" (at 0 3.2) (layer "F.Fab")
-        (effects (font (size 1 1) (thickness 0.15)))
-    )
-    (fp_text user "${REFERENCE}" (at 0 0) (layer "F.Fab")
-        (effects (font (size 1 1) (thickness 0.15)))
-    )
-    (fp_circle (center 0 0) (end 2.2 0)
-      (stroke (width 0.15) (type solid)) (fill none) (layer "Cmts.User"))
-    (fp_circle (center 0 0) (end 2.45 0)
-      (stroke (width 0.05) (type solid)) (fill none) (layer "F.CrtYd"))
-    (pad "" np_thru_hole circle (at 0 0) (size 2.2 2.2) (drill 2.2) (layers "*.Cu" "*.Mask"))
-  )
   (footprint "Resistor_SMD:R_0603_1608Metric" (layer "F.Cu")
     (at 177.860692 106.099764)
@@
     )
   )
-  (footprint "MountingHole:MountingHole_2.2mm_M2" (layer "F.Cu")
-    (at 247.071228 71.783572 90)
-    (descr "Mounting Hole 2.2mm, no annular, M2")
-    (tags "mounting hole 2.2mm no annular m2")
-    (property "Sheetfile" "disp_v8.kicad_sch")
-    (property "Sheetname" "")
-    (property "dnp" "")
-    (property "exclude_from_bom" "")
-    (property "ki_description" "Mounting Hole without connection")
-    (property "ki_keywords" "mounting hole")
-    (attr exclude_from_pos_files exclude_from_bom)
-    (fp_text reference "H2" (at 0 -3.2 90) (layer "F.SilkS") hide
-        (effects (font (size 1 1) (thickness 0.15)))
-    )
-    (fp_text value "M2" (at 0 3.2 90) (layer "F.Fab") hide
-        (effects (font (size 1 1) (thickness 0.15)))
-    )
-    (fp_text user "${REFERENCE}" (at 0 0 90) (layer "F.Fab")
-        (effects (font (size 1 1) (thickness 0.15)))
-    )
-    (fp_circle (center 0 0) (end 2.2 0)
-      (stroke (width 0.15) (type solid)) (fill none) (layer "Cmts.User"))
-    (fp_circle (center 0 0) (end 2.45 0)
-      (stroke (width 0.05) (type solid)) (fill none) (layer "F.CrtYd"))
-    (pad "" np_thru_hole circle (at 0 0 90) (size 2.2 2.2) (drill 2.2) (layers "*.Cu" "*.Mask"))
-  )
   (footprint "LED_SMD:LED_0603_1608Metric" (layer "F.Cu")

Commit message: update disp schematics for new footprints / symbols
Parts:
- J1: footprint blinky_footprints:PinSocket_2x16_P2.54mm_Vertical_FLIP -> Connector_PinHeader_2.54mm:PinHeader_2x16_P2.54mm_Vertical; moved to B.Cu
- J2, J3: moved to B.Cu
- turned J1 to 90 degrees
- turned J2 to 180 degrees
- turned J3 to 180 degrees
