File: hardware/clock_9.4/clock_9.4.kicad_sch (KiCad schematic)
At the start: 64 parts, among them J2 Conn_01x03, J4 USB_C_Receptacle, J5 Conn_01x06_Pin, J8 Conn_01x02, Q2 S8550, Q3 S8050, U10 STM32F405RGTx, U11 AMS1117-3.3, U12 BA50DD0WHFP-TR, U14 CH340C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

Commit message: clean up simple 9.4 for new power supply
Parts:
- removed C27: 100n, Capacitor_SMD:C_0603_1608Metric, symbol Device:C_Small
- removed J5: Conn_01x06_Pin, Connector_PinHeader_2.54mm:PinHeader_1x06_P2.54mm_Vertical, symbol Connector:Conn_01x06_Pin
- removed Q2: S8550, Package_TO_SOT_SMD:SOT-23, symbol BlinkyShared:S8550
- removed Q3: S8050, Package_TO_SOT_SMD:SOT-23, symbol BlinkyShared:S8050
- removed R27, R28: 4K7, Resistor_SMD:R_0603_1608Metric, symbol Device:R_US
- removed R41, R42, R54, R56, R57, R62, R65, R66, R67, R68: 1K0, Resistor_SMD:R_0603_1608Metric, symbol Device:R_Small_US
- removed R58, R59: 1K5, Resistor_SMD:R_0603_1608Metric, symbol Device:R_Small_US
- removed S3: 147873-2, SW_147873-2, symbol BlinkyShared:147873-2
- added C1, C2, C3: 100n, Capacitor_SMD:C_0402_1005Metric, symbol Device:C_Small
- added C4: 100n, Capacitor_SMD:C_0603_1608Metric, symbol Device:C_Small
- added JP3: SolderJumper_2_Bridged, Jumper:SolderJumper-2_P1.3mm_Bridged2Bar_RoundedPad1.0x1.5mm, symbol Jumper:SolderJumper_2_Bridged
- added R1, R2: 330R, Resistor_SMD:R_0603_1608Metric, symbol Device:R_Small_US
- added R3, R4: 4K7, Resistor_SMD:R_0603_1608Metric, symbol Device:R_US
- added S2: 147873-2, SW_147873-2, symbol BlinkyShared:147873-2
- added TP1, TP10, TP11, TP2, TP3, TP4, TP5, TP6, TP7, TP8, TP9: ~, TestPoint:TestPoint_THTPad_D1.5mm_Drill0.7mm, symbol Connector:TestPoint
- added U1, U2, U3: SN74LVC1G14DBV, Package_TO_SOT_SMD:SOT-23-5, symbol 74xGxx:SN74LVC1G14DBV
Connections:
- net +3.3V: now also S1.2, C1.1, C2.1, C3.1, R4.1, TP7.1, U1.5 (VCC), U2.5 (VCC), U3.5 (VCC)
- net +5V: now also TP9.1
- net +5VA: now also TP6.1
- net +6V: now also JP3.1 (A), TP5.1; no longer C44.1, JP5.2 (B), U12.2 (VCC)
- net BOOT0: now also JP1.2 (B), S1.1, R3.1, TP3.1; no longer JP2.1 (A)
- net GND: now also C1.2, C2.2, C3.2, C4.2, R3.2, S2.2, TP10.1, TP11.1, U1.3 (GND), U2.3 (GND), U3.3 (GND); no longer S1.2
- net NRST: now also JP2.2 (B), C4.1, R4.2, S2.1, TP4.1; no longer JP1.1 (A), S1.1
- net USB_DTR: now also TP1.1, U1.2
- net USB_RTS: now also TP2.1, U2.2
- new net: C44.1, JP3.2 (B), JP5.2 (B), TP8.1, U12.2 (VCC)
- new net: U1.4, U3.2
- new net: R2.2, U3.4
- new net: R1.1, U2.4
- new net: JP1.1 (A), R1.2
- new net: JP2.1 (A), R2.1
- no-connect marks 28 -> 30
Other:
- moved on the sheet: J2

Commit message: do v9.4 board with new power reg
Parts:
- removed C30: 100n, Capacitor_SMD:C_0402_1005Metric, symbol Device:C_Small
- removed C42, C44: 33u, Capacitor_Tantalum_SMD:CP_EIA-3528-21_Kemet-B, symbol Device:C_Polarized
- removed JP5: SolderJumper_2_Open, Jumper:SolderJumper-2_P1.3mm_Open_RoundedPad1.0x1.5mm, symbol Jumper:SolderJumper_2_Open
- removed U12: BA50DD0WHFP-TR, DPAK172P1054X200-6N, symbol BlinkyShared:BA50DD0WHFP-TR
- added C? (x2): 10u, Capacitor_SMD:C_0603_1608Metric, symbol Device:C_Small
- added JP5: SolderJumper_2_Bridged, Jumper:SolderJumper-2_P1.3mm_Bridged2Bar_RoundedPad1.0x1.5mm, symbol Jumper:SolderJumper_2_Bridged
- added R5: 274K, Resistor_SMD:R_0603_1608Metric, symbol Device:R_Small_US
- added R6: 30K, Resistor_SMD:R_0603_1608Metric, symbol Device:R_Small_US
- added U4: TPS7A7001DDA, Package_SO:TI_SO-PowerPAD-8, symbol Regulator_Linear:TPS7A7001DDA
Connections:
- net +5V: now also JP5.2 (B); no longer JP4.2 (B)
- net GND: now also C?.2, C?.2, R6.2, U4.8 (GND), U4.9 (EP)
- net at JP4.1 (A): now also R69.1, U4.2 (EN)
- net at JP3.2 (B), TP8.1: now also JP4.2 (B), C?.1, U4.3 (IN)
- net GPS_PPS: no longer names the net of U10.29 (PB10)
- net MON_PPS: no longer names the net of U10.30 (PB11)
- net SCL: no longer names the net of U10.61 (PB8)
- net SDA: no longer names the net of U10.62 (PB9)
- new net: C?.1, JP5.1 (A), R5.1, U4.6 (OUT)
- new net: R5.2, R6.1, U4.7 (FB)
- no-connect marks 30 -> 48
Other:
- moved on the sheet: JP3, R69, TP10, TP11, TP8

Commit message: submitted version of 9.4 board
Parts:
- J2: JLCPCB Rotation Offset (none) -> 180
- R5: value 274K -> 270K; JLCPCB Part # (none) -> C22966
- R6: JLCPCB Part # (none) -> C22984
- U4: JLCPCB Rotation Offset (none) -> 270
Other:
- note added: "270K + 30K with FB of 0.5 V gives 5V"
Changed lines of the file:
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@@
     (effects (font (size 1.27 1.27)) (justify right bottom))
   )
+  (text "270K + 30K with FB \nof 0.5 V gives 5V" (at 113.03 180.34 0)
+    (effects (font (size 1 1)) (justify left bottom))
+  )
   (label "SYNC_IN" (at 213.36 83.82 0) (fields_autoplaced)
     (effects (font (size 1.27 1.27)) (justify left bottom))
@@
       (effects (font (size 1.27 1.27)) hide)
     )
+    (property "JLCPCB Rotation Offset" "270" (at 82.55 168.91 0)
+      (effects (font (size 1.27 1.27)) hide)
+    )
     (pin "1")
     (pin "2")
@@
       (effects (font (size 1.27 1.27)) hide)
     )
+    (property "JLCPCB Rotation Offset" "180" (at 60.96 86.36 0)
+      (effects (font (size 1.27 1.27)) hide)
+    )
     (pin "1")
     (pin "2")
@@
       (effects (font (size 1.27 1.27)) hide)
     )
-    (property "LCSC" "" (at 100.33 175.26 0)
-      (effects (font (size 1.27 1.27)) hide)
-    )
-    (property "JLCPCB Part #" "" (at 100.33 175.26 0)
+    (property "JLCPCB Part #" "C22984" (at 100.33 175.26 0)
       (effects (font (size 1.27 1.27)) hide)
     )
@@
       (effects (font (size 1.27 1.27)))
     )
-    (property "Value" "274K" (at 104.14 170.18 90)
+    (property "Value" "270K" (at 104.14 170.18 90)
       (effects (font (size 1.27 1.27)))
     )
@@
       (effects (font (size 1.27 1.27)) hide)
     )
-    (property "LCSC" "" (at 100.33 168.91 0)
-      (effects (font (size 1.27 1.27)) hide)
-    )
-    (property "JLCPCB Part #" "" (at 100.33 168.91 0)
+    (property "JLCPCB Part #" "C22966" (at 100.33 168.91 0)
       (effects (font (size 1.27 1.27)) hide)
     )

Commit message: fix clock 9.4 for rotations that JLCPCB found after I submitted
Parts:
- U1, U2, U3: JLCPCB Rotation Offset 180 -> 0
Changed lines of the file:
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@@
       (effects (font (size 1.27 1.27)) hide)
     )
-    (property "JLCPCB Rotation Offset" "180" (at 304.8 137.16 0)
+    (property "JLCPCB Rotation Offset" "0" (at 304.8 137.16 0)
       (effects (font (size 1.27 1.27)) hide)
     )
@@
       (effects (font (size 1.27 1.27)) hide)
     )
-    (property "JLCPCB Rotation Offset" "180" (at 332.74 137.16 0)
+    (property "JLCPCB Rotation Offset" "0" (at 332.74 137.16 0)
       (effects (font (size 1.27 1.27)) hide)
     )
@@
       (effects (font (size 1.27 1.27)) hide)
     )
-    (property "JLCPCB Rotation Offset" "180" (at 314.96 115.57 0)
-      (effects (font (size 1.27 1.27)) hide)
-    )
+    (property "JLCPCB Rotation Offset" "0" (at 314.96 115.57 0)
+      (effects (font (size 1.27 1.27)) hide)
+    )
