File: hardware/disp_v10.0/disp_v10.0.kicad_pcb (KiCad board)
At the start: 2 copper layers, 82 x 52 mm, 115 parts, among them J1 Conn_02x16_Odd_Even_FLIP, J2 Conn_01x01_Pin, J3 Conn_01x01_Pin, Q1 2N7002, Q10 2N7002, Q11 2N7002, Q12 2N7002, Q13 2N7002, Q2 2N7002, Q3 2N7002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

Commit message: change LEDMY to LEDMB. Fixes #230
Connections:
- net /LEDMY renamed /LEDMB

Commit message: version submitted of disp v10.0 hardware
Parts:
- R1, R2, R49, R50, R51, R52, R53, R55, R56, R57: value 82R -> 100R
Changed lines of the file:
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@@
   (title_block
     (title "Disp")
-    (date "2024-01-09")
+    (date "2024-01-27")
     (rev "V10.0")
     (company "Cullen Jennings")
@@
     (descr "Resistor SMD 0603 (1608 Metric), square (rectangular) end terminal, IPC_7351 nominal, (Body size source: IPC-SM-782 page 72, https://www.pcb-3d.com/wordpress/wp-content/uploads/ipc-sm-782a_amendment_1_and_2.pdf), generated with kicad-footprint-generator")
     (tags "resistor")
-    (property "JLCPCB Part #" "C23255")
+    (property "JLCPCB Part #" "C22775")
     (property "LCSC" "")
     (property "Sheetfile" "disp_v10.0.kicad_sch")
@@
         (effects (font (size 1 1) (thickness 0.15)))
     )
-    (fp_text value "82R" (at 0 1.43 90) (layer "F.Fab")
+    (fp_text value "100R" (at 0 1.43 90) (layer "F.Fab")
         (effects (font (size 1 1) (thickness 0.15)))
     )
@@
     (descr "Resistor SMD 0603 (1608 Metric), square (rectangular) end terminal, IPC_7351 nominal, (Body size source: IPC-SM-782 page 72, https://www.pcb-3d.com/wordpress/wp-content/uploads/ipc-sm-782a_amendment_1_and_2.pdf), generated with kicad-footprint-generator")
     (tags "resistor")
-    (property "JLCPCB Part #" "C23255")
+    (property "JLCPCB Part #" "C22775")
     (property "LCSC" "")
     (property "Sheetfile" "disp_v10.0.kicad_sch")
@@
         (effects (font (size 1 1) (thickness 0.15)))
     )
-    (fp_text value "82R" (at 0 1.43 90) (layer "F.Fab")
+    (fp_text value "100R" (at 0 1.43 90) (layer "F.Fab")
         (effects (font (size 1 1) (thickness 0.15)))
     )
@@
     (descr "Resistor SMD 0603 (1608 Metric), square (rectangular) end terminal, IPC_7351 nominal, (Body size source: IPC-SM-782 page 72, https://www.pcb-3d.com/wordpress/wp-content/uploads/ipc-sm-782a_amendment_1_and_2.pdf), generated with kicad-footprint-generator")
     (tags "resistor")
-    (property "JLCPCB Part #" "C23255")
+    (property "JLCPCB Part #" "C22775")
     (property "LCSC" "")
     (property "Sheetfile" "disp_v10.0.kicad_sch")
@@
         (effects (font (size 1 1) (thickness 0.15)))
     )
-    (fp_text value "82R" (at 0 1.43 90) (layer "F.Fab")
+    (fp_text value "100R" (at 0 1.43 90) (layer "F.Fab")
         (effects (font (size 1 1) (thickness 0.15)))
     )
@@
     (descr "Resistor SMD 0603 (1608 Metric), square (rectangular) end terminal, IPC_7351 nominal, (Body size source: IPC-SM-782 page 72, https://www.pcb-3d.com/wordpress/wp-content/uploads/ipc-sm-782a_amendment_1_and_2.pdf), generated with kicad-footprint-generator")
     (tags "resistor")
-    (property "JLCPCB Part #" "C23255")
+    (property "JLCPCB Part #" "C22775")
     (property "LCSC" "")
     (property "Sheetfile" "disp_v10.0.kicad_sch")
@@
         (effects (font (size 1 1) (thickness 0.15)))
     )
-    (fp_text value "82R" (at 0 1.43 90) (layer "F.Fab")
+    (fp_text value "100R" (at 0 1.43 90) (layer "F.Fab")
         (effects (font (size 1 1) (thickness 0.15)))
     )
@@
     (descr "Resistor SMD 0603 (1608 Metric), square (rectangular) end terminal, IPC_7351 nominal, (Body size source: IPC-SM-782 page 72, https://www.pcb-3d.com/wordpress/wp-content/uploads/ipc-sm-782a_amendment_1_and_2.pdf), generated with kicad-footprint-generator")
     (tags "resistor")
-    (property "JLCPCB Part #" "C23255")
+    (property "JLCPCB Part #" "C22775")
     (property "LCSC" "")
     (property "Sheetfile" "disp_v10.0.kicad_sch")
@@
         (effects (font (size 1 1) (thickness 0.15)))
     )
-    (fp_text value "82R" (at 0 1.43 90) (layer "F.Fab")
+    (fp_text value "100R" (at 0 1.43 90) (layer "F.Fab")
         (effects (font (size 1 1) (thickness 0.15)))
     )
@@
     (descr "Resistor SMD 0603 (1608 Metric), square (rectangular) end terminal, IPC_7351 nominal, (Body size source: IPC-SM-782 page 72, https://www.pcb-3d.com/wordpress/wp-content/uploads/ipc-sm-782a_amendment_1_and_2.pdf), generated with kicad-footprint-generator")
     (tags "resistor")
-    (property "JLCPCB Part #" "C23255")
+    (property "JLCPCB Part #" "C22775")
     (property "LCSC" "")
     (property "Sheetfile" "disp_v10.0.kicad_sch")
@@
         (effects (font (size 1 1) (thickness 0.15)))
     )
-    (fp_text value "82R" (at 0 1.43 90) (layer "F.Fab")
+    (fp_text value "100R" (at 0 1.43 90) (layer "F.Fab")
         (effects (font (size 1 1) (thickness 0.15)))
     )
@@
     (descr "Resistor SMD 0603 (1608 Metric), square (rectangular) end terminal, IPC_7351 nominal, (Body size source: IPC-SM-782 page 72, https://www.pcb-3d.com/wordpress/wp-content/uploads/ipc-sm-782a_amendment_1_and_2.pdf), generated with kicad-footprint-generator")
     (tags "resistor")
-    (property "JLCPCB Part #" "C23255")
+    (property "JLCPCB Part #" "C22775")
     (property "LCSC" "")
     (property "Sheetfile" "disp_v10.0.kicad_sch")
@@
         (effects (font (size 1 1) (thickness 0.15)))
     )
-    (fp_text value "82R" (at 0 1.43 90) (layer "F.Fab")
+    (fp_text value "100R" (at 0 1.43 90) (layer "F.Fab")
         (effects (font (size 1 1) (thickness 0.15)))
     )
@@
     (descr "Resistor SMD 0603 (1608 Metric), square (rectangular) end terminal, IPC_7351 nominal, (Body size source: IPC-SM-782 page 72, https://www.pcb-3d.com/wordpress/wp-content/uploads/ipc-sm-782a_amendment_1_and_2.pdf), generated with kicad-footprint-generator")
     (tags "resistor")
-    (property "JLCPCB Part #" "C23255")
+    (property "JLCPCB Part #" "C22775")
     (property "LCSC" "")
     (property "Sheetfile" "disp_v10.0.kicad_sch")
@@
         (effects (font (size 1 1) (thickness 0.15)))
     )
-    (fp_text value "82R" (at 0 1.43 90) (layer "F.Fab")
+    (fp_text value "100R" (at 0 1.43 90) (layer "F.Fab")
         (effects (font (size 1 1) (thickness 0.15)))
     )
@@
     (descr "Resistor SMD 0603 (1608 Metric), square (rectangular) end terminal, IPC_7351 nominal, (Body size source: IPC-SM-782 page 72, https://www.pcb-3d.com/wordpress/wp-content/uploads/ipc-sm-782a_amendment_1_and_2.pdf), generated with kicad-footprint-generator")
     (tags "resistor")
-    (property "JLCPCB Part #" "C23255")
+    (property "JLCPCB Part #" "C22775")
     (property "LCSC" "")
     (property "Sheetfile" "disp_v10.0.kicad_sch")
@@
         (effects (font (size 1 1) (thickness 0.15)))
     )
-    (fp_text value "82R" (at 0 1.43 90) (layer "F.Fab")
+    (fp_text value "100R" (at 0 1.43 90) (layer "F.Fab")
         (effects (font (size 1 1) (thickness 0.15)))
     )
@@
     (descr "Resistor SMD 0603 (1608 Metric), square (rectangular) end terminal, IPC_7351 nominal, (Body size source: IPC-SM-782 page 72, https://www.pcb-3d.com/wordpress/wp-content/uploads/ipc-sm-782a_amendment_1_and_2.pdf), generated with kicad-footprint-generator")
     (tags "resistor")
-    (property "JLCPCB Part #" "C23255")
+    (property "JLCPCB Part #" "C22775")
     (property "LCSC" "")
     (property "Sheetfile" "disp_v10.0.kicad_sch")
@@
         (effects (font (size 1 1) (thickness 0.15)))
     )
-    (fp_text value "82R" (at 0 1.43 90) (layer "F.Fab")
+    (fp_text value "100R" (at 0 1.43 90) (layer "F.Fab")
         (effects (font (size 1 1) (thickness 0.15)))
     )
