File: hardware/disp_v10.0/disp_v10.0.kicad_sch (KiCad schematic)
At the start: 115 parts, among them J1 Conn_02x16_Odd_Even_FLIP, J2 Conn_01x01_Pin, J3 Conn_01x01_Pin, Q1 2N7002, Q10 2N7002, Q11 2N7002, Q12 2N7002, Q13 2N7002, Q2 2N7002, Q3 2N7002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

Commit message: change LEDMY to LEDMB. Fixes #230
Connections:
- net LEDMY renamed LEDMB
Changed lines of the file:
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@@
     (effects (font (size 1.27 1.27)) (justify left bottom))
   )
-  (label "LEDMY" (at 48.26 31.75 0) (fields_autoplaced)
+  (label "LEDMB" (at 48.26 31.75 0) (fields_autoplaced)
     (effects (font (size 1.27 1.27)) (justify left bottom))
   )
-  (label "LEDMY" (at 100.33 72.39 0) (fields_autoplaced)
+  (label "LEDMB" (at 100.33 72.39 0) (fields_autoplaced)
     (effects (font (size 1.27 1.27)) (justify left bottom))
   )

Commit message: version submitted of disp v10.0 hardware
Parts:
- R1, R2, R49, R50, R51, R52, R53, R55, R56, R57: value 82R -> 100R; JLCPCB Part # C23255 -> C22775
Changed lines of the file:
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@@
   (title_block
     (title "Disp")
-    (date "2024-01-09")
+    (date "2024-01-27")
     (rev "V10.0")
     (company "Cullen Jennings")
@@
       (effects (font (size 1.27 1.27)))
     )
-    (property "Value" "82R" (at 184.15 21.59 90)
+    (property "Value" "100R" (at 184.15 21.59 90)
       (effects (font (size 1.27 1.27)))
     )
@@
       (effects (font (size 1.27 1.27)) hide)
     )
-    (property "JLCPCB Part #" "C23255" (at 184.15 25.4 0)
+    (property "JLCPCB Part #" "C22775" (at 184.15 25.4 0)
       (effects (font (size 1.27 1.27)) hide)
     )
@@
       (effects (font (size 1.27 1.27)))
     )
-    (property "Value" "82R" (at 184.15 45.72 90)
+    (property "Value" "100R" (at 184.15 45.72 90)
       (effects (font (size 1.27 1.27)))
     )
@@
       (effects (font (size 1.27 1.27)) hide)
     )
-    (property "JLCPCB Part #" "C23255" (at 184.15 49.53 0)
+    (property "JLCPCB Part #" "C22775" (at 184.15 49.53 0)
       (effects (font (size 1.27 1.27)) hide)
     )
@@
       (effects (font (size 1.27 1.27)))
     )
-    (property "Value" "82R" (at 184.15 88.9 90)
+    (property "Value" "100R" (at 184.15 88.9 90)
       (effects (font (size 1.27 1.27)))
     )
@@
       (effects (font (size 1.27 1.27)) hide)
     )
-    (property "JLCPCB Part #" "C23255" (at 184.15 92.71 0)
+    (property "JLCPCB Part #" "C22775" (at 184.15 92.71 0)
       (effects (font (size 1.27 1.27)) hide)
     )
@@
       (effects (font (size 1.27 1.27)))
     )
-    (property "Value" "82R" (at 184.15 33.02 90)
+    (property "Value" "100R" (at 184.15 33.02 90)
       (effects (font (size 1.27 1.27)))
     )
@@
       (effects (font (size 1.27 1.27)) hide)
     )
-    (property "JLCPCB Part #" "C23255" (at 184.15 36.83 0)
+    (property "JLCPCB Part #" "C22775" (at 184.15 36.83 0)
       (effects (font (size 1.27 1.27)) hide)
     )
@@
       (effects (font (size 1.27 1.27)))
     )
-    (property "Value" "82R" (at 184.15 59.69 90)
+    (property "Value" "100R" (at 184.15 59.69 90)
       (effects (font (size 1.27 1.27)))
     )
@@
       (effects (font (size 1.27 1.27)) hide)
     )
-    (property "JLCPCB Part #" "C23255" (at 184.15 63.5 0)
+    (property "JLCPCB Part #" "C22775" (at 184.15 63.5 0)
       (effects (font (size 1.27 1.27)) hide)
     )
@@
       (effects (font (size 1.27 1.27)))
     )
-    (property "Value" "82R" (at 182.88 133.35 90)
+    (property "Value" "100R" (at 182.88 133.35 90)
       (effects (font (size 1.27 1.27)))
     )
@@
       (effects (font (size 1.27 1.27)) hide)
     )
-    (property "JLCPCB Part #" "C23255" (at 182.88 137.16 0)
+    (property "JLCPCB Part #" "C22775" (at 182.88 137.16 0)
       (effects (font (size 1.27 1.27)) hide)
     )
@@
       (effects (font (size 1.27 1.27)))
     )
-    (property "Value" "82R" (at 182.88 147.32 90)
+    (property "Value" "100R" (at 182.88 147.32 90)
       (effects (font (size 1.27 1.27)))
     )
@@
       (effects (font (size 1.27 1.27)) hide)
     )
-    (property "JLCPCB Part #" "C23255" (at 182.88 151.13 0)
+    (property "JLCPCB Part #" "C22775" (at 182.88 151.13 0)
       (effects (font (size 1.27 1.27)) hide)
     )
@@
       (effects (font (size 1.27 1.27)))
     )
-    (property "Value" "82R" (at 184.15 105.41 90)
+    (property "Value" "100R" (at 184.15 105.41 90)
       (effects (font (size 1.27 1.27)))
     )
@@
       (effects (font (size 1.27 1.27)) hide)
     )
-    (property "JLCPCB Part #" "C23255" (at 184.15 109.22 0)
+    (property "JLCPCB Part #" "C22775" (at 184.15 109.22 0)
       (effects (font (size 1.27 1.27)) hide)
     )
@@
       (effects (font (size 1.27 1.27)))
     )
-    (property "Value" "82R" (at 184.15 73.66 90)
+    (property "Value" "100R" (at 184.15 73.66 90)
       (effects (font (size 1.27 1.27)))
     )
@@
       (effects (font (size 1.27 1.27)) hide)
     )
-    (property "JLCPCB Part #" "C23255" (at 184.15 77.47 0)
+    (property "JLCPCB Part #" "C22775" (at 184.15 77.47 0)
       (effects (font (size 1.27 1.27)) hide)
     )
@@
       (effects (font (size 1.27 1.27)))
     )
-    (property "Value" "82R" (at 184.15 119.38 90)
+    (property "Value" "100R" (at 184.15 119.38 90)
       (effects (font (size 1.27 1.27)))
     )
@@
       (effects (font (size 1.27 1.27)) hide)
     )
-    (property "JLCPCB Part #" "C23255" (at 184.15 123.19 0)
+    (property "JLCPCB Part #" "C22775" (at 184.15 123.19 0)
       (effects (font (size 1.27 1.27)) hide)
     )
