File: hardware/gps_v12/gps_v12.kicad_sch (KiCad schematic)
At the start: 90 parts, among them J1 RJ45, J4 USB_C_Receptacle, Q1 2N7002, Q10 2N7002, Q9 2N7002, U10 STM32F405RGTx, U11 AMS1117-3.3, U13 M24C02-RMN, U14 CH340C, U15 USBLC6-2P6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

Commit message: add 3d model for RJ45 connector
Parts:
- J1: footprint Connector_RJ:RJ45_Amphenol_RJHSE5380 -> blinky_footprints:RJ45_Amphenol_RJHSE5380
- J4: footprint Connector_USB:USB_C_Receptacle_HRO_TYPE-C-31-M-12 -> blinky_footprints:USB_C_Receptacle_HRO_TYPE-C-31-M-12
Changed lines of the file:
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@@
 			)
 		)
-		(property "Footprint" "Connector_USB:USB_C_Receptacle_HRO_TYPE-C-31-M-12"
+		(property "Footprint" "blinky_footprints:USB_C_Receptacle_HRO_TYPE-C-31-M-12"
 			(at 135.89 190.5 0)
 			(effects
@@
 			)
 		)
-		(property "Footprint" "Connector_RJ:RJ45_Amphenol_RJHSE5380"
+		(property "Footprint" "blinky_footprints:RJ45_Amphenol_RJHSE5380"
 			(at 30.48 247.015 90)
 			(effects
