File: hardware/blink_v13/blink_v13.kicad_pcb (KiCad board)
At the start: 2 copper layers, 119 x 92 mm, 164 parts, among them J1 Conn_01x02, J11 KH-BNC50-3511, J12 KH-BNC50-3511, J13 KH-BNC50-3511, J14 Conn_02x16_Odd_Even, J15 Conn_01x01, J16 Conn_01x01, J2 PJ-320D, J3 PJ-320D, J4 KH-BNC50-3511, J5 Conn_01x06_Pin, J6 Conn_01x03, J7 Conn_01x06_Pin, J9 USB_C_Receptacle, Q3 2N7002, Q4 2N7002, Q5 2N7002, SW1 SW_SPDT, SW2 SW_Push_4PDT, SW3 SW_Push_4PDT, SW4 SW_Push_4PDT, U1 AMS1117-3.3, U10 TMP112AIDRLR, U11 MAX40200AUK, U12 MAX40200AUK, U13 AMS1117-3.3, U14 SN74LVC1G14DBV, U16 TPS63060, U2 AD8397, U3 M24C02-RMN, U4 STM32F405RGTx, U5 SN74LVC1G14DBV, U6 SN74LVC1G14DBV, U7 CH340C, U8 USBLC6-2P6, U9 MCP73832-2-OT, X1 GTXO-14V (2.048MHz), Y1 16MHz

Commit message: clean up version for blink v13
Other:
- board text added: "Blink V13 Cullen Jennings"
- board text removed: "Blink V12 Cullen Jennings"
Changed lines of the file:
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@@
 	(title_block
 		(title "Blink")
-		(date "2024-04-03")
-		(rev "V12")
+		(date "2024-04-10")
+		(rev "V13")
 		(company "Cullen Jennings")
 	)
@@
 		(tags "capacitor")
 		(property "Reference" "C3"
-			(at 0 -1.43 270)
+			(at 0 -1.43 -90)
 			(layer "F.SilkS")
 			(hide yes)
@@
 		)
 		(property "Value" "10u"
-			(at 0 1.43 270)
+			(at 0 1.43 -90)
 			(layer "F.Fab")
 			(effects
@@
 		)
 		(fp_text user "${REFERENCE}"
-			(at 0 0 270)
+			(at 0 0 -90)
 			(layer "F.Fab")
 			(effects
@@
 		(layer "Edge.Cuts")
 	)
-	(gr_text "Blink V12 Cullen Jennings "
+	(gr_text "Blink V13 Cullen Jennings "
 		(at 175.22069 41.354948 0)
 		(layer "F.SilkS")
