File: hardware/gps_A/gps_A.kicad_sch (KiCad schematic)
At the start: 90 parts, among them J1 RJ45, J4 USB_C_Receptacle, Q1 2N7002, Q10 2N7002, Q9 2N7002, U10 STM32F405RGTx, U11 AMS1117-3.3, U13 M24C02-RMN, U14 CH340C, U15 USBLC6-2P6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

Commit message: start generation of GPS rev A.1 production files
Parts:
- D4: value SDM20U30-7 -> B5819W SL; footprint Diode_SMD:D_SOD-523 -> Diode_SMD:D_SOD-123; JLCPCB Part # C91235 -> C8598
- J1: footprint Connector_RJ:RJ45_Amphenol_RJHSE5380 -> blinky_footprints:RJ45_Amphenol_RJHSE5380
- J4: footprint Connector_USB:USB_C_Receptacle_HRO_TYPE-C-31-M-12 -> blinky_footprints:USB_C_Receptacle_HRO_TYPE-C-31-M-12; JLCPCB Position Offset 0,1.3 -> 0,1.1
- U8: footprint SC70_DCK_TEX -> blinky_footprints:SC70_DCK_TEX
Connections:
- net at J4.A6 (D+), J4.B6 (D+): now also U15.1 (I/O1); no longer U15.6 (I/O1)
- net at J4.A7 (D-), J4.B7 (D-): now also U15.6 (I/O1); no longer U15.4 (I/O2)
- net at U14.5 (UD+): now also U15.3 (I/O2); no longer U15.1 (I/O1)
- net at U14.6 (UD-): now also U15.4 (I/O2); no longer U15.3 (I/O2)
- no-connect marks 37 -> 40
Other:
- moved on the sheet: C57, C58, D4

Commit message: version of GPS Rev A.1  submitted to JLCPCB
Connections:
- net at J4.A6 (D+), J4.B6 (D+): now also U15.6 (I/O1); no longer U15.1 (I/O1)
- net at J4.A7 (D-), J4.B7 (D-): now also U15.4 (I/O2); no longer U15.6 (I/O1)
- net at U14.5 (UD+): now also U15.1 (I/O1); no longer U15.3 (I/O2)
- net at U14.6 (UD-): now also U15.3 (I/O2); no longer U15.4 (I/O2)
Other:
- moved on the sheet: U15
Changed lines of the file:
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@@
 	(wire
 		(pts
-			(xy 76.2 185.42) (xy 96.52 185.42)
-		)
-		(stroke
-			(width 0)
-			(type default)
-		)
-	)
-	(wire
-		(pts
 			(xy 275.59 31.75) (xy 275.59 35.56)
 		)
@@
 	(wire
 		(pts
+			(xy 73.66 182.88) (xy 73.66 184.15)
+		)
+		(stroke
+			(width 0)
+			(type default)
+		)
+	)
+	(wire
+		(pts
 			(xy 504.19 139.7) (xy 504.19 142.24)
 		)
@@
 	(wire
 		(pts
-			(xy 59.69 189.23) (xy 55.88 189.23)
+			(xy 55.88 189.23) (xy 68.58 189.23)
 		)
 		(stroke
@@
 	(wire
 		(pts
-			(xy 59.69 185.42) (xy 59.69 189.23)
-		)
-		(stroke
-			(width 0)
-			(type default)
-		)
-	)
-	(wire
-		(pts
 			(xy 35.56 199.39) (xy 25.4 199.39)
 		)
@@
 	(wire
 		(pts
-			(xy 438.15 86.36) (xy 443.23 86.36)
+			(xy 73.66 196.85) (xy 73.66 198.12)
 		)
 		(stroke
@@
 	(wire
 		(pts
-			(xy 99.06 205.74) (xy 99.06 165.1)
+			(xy 438.15 86.36) (xy 443.23 86.36)
 		)
 		(stroke
@@
 	(wire
 		(pts
-			(xy 96.52 185.42) (xy 96.52 162.56)
+			(xy 96.52 162.56) (xy 96.52 189.23)
 		)
 		(stroke
@@
 	(wire
 		(pts
-			(xy 44.45 252.73) (xy 44.45 256.54)
+			(xy 78.74 189.23) (xy 96.52 189.23)
 		)
 		(stroke
@@
 	(wire
 		(pts
-			(xy 227.33 49.53) (xy 229.87 49.53)
+			(xy 44.45 252.73) (xy 44.45 256.54)
 		)
 		(stroke
@@
 	(wire
 		(pts
-			(xy 207.01 58.42) (xy 217.17 58.42)
+			(xy 227.33 49.53) (xy 229.87 49.53)
 		)
 		(stroke
@@
 	(wire
 		(pts
-			(xy 63.5 254) (xy 63.5 260.35)
+			(xy 207.01 58.42) (xy 217.17 58.42)
 		)
 		(stroke
@@
 	(wire
 		(pts
-			(xy 204.47 232.41) (xy 209.55 232.41)
+			(xy 63.5 254) (xy 63.5 260.35)
 		)
 		(stroke
@@
 	(wire
 		(pts
-			(xy 297.18 292.1) (xy 299.72 292.1)
+			(xy 204.47 232.41) (xy 209.55 232.41)
 		)
 		(stroke
@@
 	(wire
 		(pts
-			(xy 135.89 177.8) (xy 115.57 177.8)
+			(xy 297.18 292.1) (xy 299.72 292.1)
 		)
 		(stroke
@@
 	(wire
 		(pts
-			(xy 76.2 200.66) (xy 76.2 205.74)
+			(xy 135.89 177.8) (xy 115.57 177.8)
 		)
 		(stroke
@@
 	(wire
 		(pts
-			(xy 76.2 185.42) (xy 76.2 190.5)
-		)
-		(stroke
-			(width 0)
-			(type default)
-		)
-	)
-	(wire
-		(pts
 			(xy 270.51 130.81) (xy 269.24 130.81)
 		)
@@
 	(wire
 		(pts
-			(xy 81.28 195.58) (xy 90.17 195.58)
-		)
-		(stroke
-			(width 0)
-			(type default)
-		)
-	)
-	(wire
-		(pts
 			(xy 215.9 295.91) (xy 259.08 295.91)
 		)
@@
 	(wire
 		(pts
+			(xy 99.06 191.77) (xy 99.06 165.1)
+		)
+		(stroke
+			(width 0)
+			(type default)
+		)
+	)
+	(wire
+		(pts
 			(xy 267.97 130.81) (xy 267.97 129.54)
 		)
@@
 	(wire
 		(pts
-			(xy 55.88 191.77) (xy 59.69 191.77)
+			(xy 55.88 191.77) (xy 68.58 191.77)
 		)
 		(stroke
@@
 	(wire
 		(pts
-			(xy 86.36 300.99) (xy 87.63 300.99)
+			(xy 78.74 191.77) (xy 99.06 191.77)
 		)
 		(stroke
@@
 	(wire
 		(pts
-			(xy 265.43 31.75) (xy 265.43 35.56)
+			(xy 86.36 300.99) (xy 87.63 300.99)
 		)
 		(stroke
@@
 	(wire
 		(pts
-			(xy 73.66 185.42) (xy 73.66 190.5)
+			(xy 265.43 31.75) (xy 265.43 35.56)
 		)
 		(stroke
@@
 	(wire
 		(pts
-			(xy 73.66 185.42) (xy 59.69 185.42)
-		)
-		(stroke
-			(width 0)
-			(type default)
-		)
-	)
-	(wire
-		(pts
 			(xy 55.88 73.66) (xy 67.31 73.66)
 		)
@@
 	(wire
 		(pts
-			(xy 59.69 191.77) (xy 59.69 205.74)
-		)
-		(stroke
-			(width 0)
-			(type default)
-		)
-	)
-	(wire
-		(pts
 			(xy 270.51 31.75) (xy 270.51 35.56)
 		)
@@
 	(wire
 		(pts
-			(xy 73.66 200.66) (xy 73.66 205.74)
-		)
-		(stroke
-			(width 0)
-			(type default)
-		)
-	)
-	(wire
-		(pts
 			(xy 510.54 142.24) (xy 504.19 142.24)
 		)
@@
 	(wire
 		(pts
-			(xy 59.69 205.74) (xy 73.66 205.74)
-		)
-		(stroke
-			(width 0)
-			(type default)
-		)
-	)
-	(wire
-		(pts
 			(xy 502.92 132.08) (xy 504.19 132.08)
 		)
@@
 	(wire
 		(pts
-			(xy 66.04 195.58) (xy 68.58 195.58)
-		)
-		(stroke
-			(width 0)
-			(type default)
-		)
-	)
-	(wire
-		(pts
 			(xy 257.81 341.63) (xy 264.16 341.63)
 		)
@@
 	(wire
 		(pts
-			(xy 76.2 205.74) (xy 99.06 205.74)
-		)
-		(stroke
-			(width 0)
-			(type default)
-		)
-	)
-	(wire
-		(pts
 			(xy 273.05 35.56) (xy 273.05 31.75)
 		)
@@
 	(symbol
 		(lib_id "power:GND")
-		(at 66.04 195.58 270)
+		(at 73.66 198.12 0)
 		(unit 1)
 		(exclude_from_sim no)
@@
 		(dnp no)
 		(property "Reference" "#PWR031"
-			(at 59.69 195.58 0)
+			(at 73.66 204.47 0)
 			(effects
 				(font
@@
 		)
 		(property "Value" "GND"
-			(at 62.23 198.12 0)
+			(at 76.2 201.93 0)
 			(effects
 				(font
@@
 		)
 		(property "Footprint" ""
-			(at 66.04 195.58 0)
+			(at 73.66 198.12 0)
 			(effects
 				(font
@@
 		)
 		(property "Datasheet" ""
-			(at 66.04 195.58 0)
+			(at 73.66 198.12 0)
 			(effects
 				(font
@@
 		)
 		(property "Description" "Power symbol creates a global label with name \"GND\" , ground"
-			(at 66.04 195.58 0)
+			(at 73.66 198.12 0)
 			(effects
 				(font
@@
 	(symbol
 		(lib_id "Power_Protection:USBLC6-2P6")
-		(at 76.2 195.58 270)
+		(at 73.66 189.23 0)
 		(unit 1)
 		(exclude_from_sim no)
@@
 		(dnp no)
 		(property "Reference" "U15"
-			(at 67.31 189.23 0)
+			(at 67.31 198.12 0)
 			(effects
 				(font
@@
 		)
 		(property "Value" "USBLC6-2P6"
-			(at 76.2 190.5 90)
+			(at 83.566 193.802 0)
 			(effects
 				(font
@@
 		)
 		(property "Footprint" "Package_TO_SOT_SMD:SOT-666"
-			(at 63.5 195.58 0)
+			(at 73.66 201.93 0)
 			(effects
 				(font
@@
 		)
 		(property "Datasheet" "https://www.st.com/resource/en/datasheet/usblc6-2.pdf"
-			(at 85.09 200.66 0)
+			(at 78.74 180.34 0)
 			(effects
 				(font
@@
 		)
 		(property "Description" "Very low capacitance ESD protection diode, 2 data-line, SOT-666"
-			(at 76.2 195.58 0)
+			(at 73.66 189.23 0)
 			(effects
 				(font
@@
 		)
 		(property "JLCPCB#" ""
-			(at 76.2 195.58 0)
+			(at 73.66 189.23 0)
 			(effects
 				(font
@@
 		)
 		(property "JLCPCB Part #" "C2827693"
-			(at 76.2 195.58 0)
+			(at 73.66 189.23 0)
 			(effects
 				(font
@@
 		)
 		(property "JLCPCB Rotation Offset" "270"
-			(at 76.2 195.58 0)
+			(at 73.66 189.23 0)
 			(effects
 				(font
@@
 	(symbol
 		(lib_id "power:VBUS")
-		(at 90.17 195.58 270)
+		(at 73.66 182.88 0)
 		(unit 1)
 		(exclude_from_sim no)
@@
 		(dnp no)
 		(property "Reference" "#PWR047"
-			(at 86.36 195.58 0)
+			(at 73.66 186.69 0)
 			(effects
 				(font
@@
 		)
 		(property "Value" "VBUS"
-			(at 92.71 198.12 90)
+			(at 76.2 180.34 90)
 			(effects
 				(font
@@
 		)
 		(property "Footprint" ""
-			(at 90.17 195.58 0)
+			(at 73.66 182.88 0)
 			(effects
 				(font
@@
 		)
 		(property "Datasheet" ""
-			(at 90.17 195.58 0)
+			(at 73.66 182.88 0)
 			(effects
 				(font
@@
 		)
 		(property "Description" "Power symbol creates a global label with name \"VBUS\""
-			(at 90.17 195.58 0)
+			(at 73.66 182.88 0)
 			(effects
 				(font

Commit message: remove tal caps on GPS, clean up schamatic
Parts:
- removed C41: 10u, Capacitor_Tantalum_SMD:CP_EIA-3216-18_Kemet-A, symbol Device:C_Polarized
- added C2: 10u, Capacitor_SMD:C_0603_1608Metric, symbol Device:C_Small
- C42: value 33u -> 10u; footprint Capacitor_Tantalum_SMD:CP_EIA-3528-21_Kemet-B -> Capacitor_SMD:C_0603_1608Metric; symbol Device:C_Polarized -> Device:C_Small; JLCPCB Part # C128342 -> C19702
Connections:
- net +3.3V: now also C2.1
- net GND: now also C2.2
- no-connect marks 40 -> 38
Other:
- note added: "Inputs"
- note added: "Status"
- note removed: "Status / Control"
- moved on the sheet: C1, C11, C27, C39, C4, C45, C47, C48, C50, C56, C57, C58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

Commit message: update rotation and offsets on clock and gps
Parts:
- D5: JLCPCB Position Offset 0,-0.75 -> 0,0.7
- J4: JLCPCB Position Offset 0,1.1 -> 0,1.5
- J?: JLCPCB Position Offset (none) -> 0,-13.0
- U10, U13, U14: JLCPCB Rotation Offset 270 -> (none)
- U11: JLCPCB Rotation Offset 180 -> (none)
- U19, U2, U20, U21: JLCPCB Rotation Offset 0 -> (none)
- U8: footprint blinky_footprints:SC70_DCK_TEX -> Package_TO_SOT_SMD:SOT-363_SC-70-6
Changed lines of the file:
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@@
 			)
 		)
-		(property "JLCPCB Rotation Offset" "0"
+		(property "JLCPCB Rotation Offset" ""
 			(at 55.88 215.9 0)
 			(effects
@@
 			)
 		)
-		(property "Footprint" "blinky_footprints:SC70_DCK_TEX"
+		(property "Footprint" "Package_TO_SOT_SMD:SOT-363_SC-70-6"
 			(at 102.87 172.72 0)
 			(effects
@@
 			)
 		)
-		(property "JLCPCB Rotation Offset" "270"
+		(property "JLCPCB Rotation Offset" ""
 			(at 267.97 83.82 0)
 			(effects
@@
 			)
 		)
-		(property "JLCPCB Position Offset" "0,1.1"
+		(property "JLCPCB Position Offset" "0,1.5"
 			(at 123.19 121.92 0)
 			(effects
@@
 			)
 		)
-		(property "JLCPCB Rotation Offset" "180"
+		(property "JLCPCB Rotation Offset" ""
 			(at 41.91 58.42 0)
 			(effects
@@
 			)
 		)
-		(property "JLCPCB Rotation Offset" "0"
+		(property "JLCPCB Rotation Offset" ""
 			(at 198.12 171.45 0)
 			(effects
@@
 			)
 		)
-		(property "JLCPCB Rotation Offset" "270"
+		(property "JLCPCB Rotation Offset" ""
 			(at 300.99 170.18 0)
 			(effects
@@
 			)
 		)
-		(property "JLCPCB Rotation Offset" "270"
+		(property "JLCPCB Rotation Offset" ""
 			(at 49.53 119.38 0)
 			(effects
@@
 			)
 		)
-		(property "JLCPCB Rotation Offset" "0"
+		(property "JLCPCB Rotation Offset" ""
 			(at 106.68 228.6 0)
 			(effects
@@
 			)
 		)
-		(property "JLCPCB Rotation Offset" "0"
+		(property "JLCPCB Rotation Offset" ""
 			(at 109.22 39.37 0)
 			(effects
@@
 			)
 		)
+		(property "JLCPCB Position Offset" "0,-13.0"
+			(at 236.22 171.45 0)
+			(effects
+				(font
+					(size 1.27 1.27)
+				)
+				(hide yes)
+			)
+		)
 		(pin "1"
 		)
@@
 			)
 		)
-		(property "JLCPCB Position Offset" "0,-0.75"
+		(property "JLCPCB Position Offset" "0,0.7"
 			(at 381 168.91 0)
 			(effects

Commit message: Update jlc part num for CH340 Fixes#346
Parts:
- U14: JLCPCB Part # C84681 -> C7464026
Changed lines of the file:
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@@
 			)
 		)
-		(property "JLCPCB Part #" "C84681"
+		(property "JLCPCB Part #" "C7464026"
 			(at 49.53 119.38 0)
 			(effects

Commit message: order GPS A.2
Parts:
- Q1, Q10, Q9: JLCPCB Rotation Offset 180 -> (none)
Changed lines of the file:
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@@
 	(title_block
 		(title "GPS")
-		(date "2024-05-27")
+		(date "2024-06-16")
 		(rev "A.2")
 		(company "Cullen Jennings")
@@
 			)
 		)
-		(property "JLCPCB Rotation Offset" "180"
+		(property "JLCPCB Rotation Offset" ""
 			(at 355.6 184.15 0)
 			(effects
@@
 			)
 		)
-		(property "JLCPCB Rotation Offset" "180"
+		(property "JLCPCB Rotation Offset" ""
 			(at 355.6 199.39 0)
 			(effects
@@
 			)
 		)
-		(property "JLCPCB Rotation Offset" "180"
+		(property "JLCPCB Rotation Offset" ""
 			(at 355.6 215.9 0)
 			(effects

Commit message: updates for GPS Rev A.3
Parts:
- removed R28: 47K, Resistor_SMD:R_0603_1608Metric, symbol Device:R_US
- removed R32: 4K7, Resistor_SMD:R_0603_1608Metric, symbol Device:R_US
- added J6: Conn_01x03, Connector_JST:JST_PH_S3B-PH-SM4-TB_1x03-1MP_P2.00mm_Horizontal, symbol Connector_Generic:Conn_01x03
- Y2: value 16MHz -> 16MHz
- gave numbers to parts that had none: 2
Connections:
- net GND: now also J6.2 (Pin_2)
- net SWDCLK: now also J6.3 (Pin_3)
- net SWDIO: now also J6.1 (Pin_1)
- no-connect marks 38 -> 36
Other:
- moved on the sheet: R22
