File: hardware/blink_A/blink_A.kicad_sch (KiCad schematic)
At the start: 166 parts, among them J1 Conn_01x02, J14 Conn_02x16_Odd_Even, J15 Conn_01x01, J16 Conn_01x01, J5 Conn_01x06_Pin, J6 Conn_01x03, J7 Conn_01x06_Pin, J9 USB_C_Receptacle, Q3 2N7002, Q4 2N7002, Q5 2N7002, SW1 SW_SPDT, SW2 SW_Push_4PDT, SW3 SW_Push_4PDT, SW4 SW_Push_4PDT, U1 AMS1117-3.3, U10 TMP112AIDRLR, U11 MAX40200AUK, U12 MAX40200AUK, U13 AMS1117-3.3, U14 SN74LVC1G14DBV, U16 TPS63060, U3 M24C02-RMN, U4 STM32F405RGTx, U5 SN74LVC1G14DBV, U6 SN74LVC1G14DBV, U7 CH340C, U8 USBLC6-2P6, U9 MCP73832-2-OT, X1 GTXO-14V (2.048MHz), Y1 16MHz

Commit message: update rotation and offsets on clock and gps
Parts:
- U14, U3, U4, U5, U6: JLCPCB Rotation Offset 0 -> (none)
Changed lines of the file:
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@@
 			)
 		)
-		(property "JLCPCB Rotation Offset" "0"
+		(property "JLCPCB Rotation Offset" ""
 			(at 229.87 88.9 0)
 			(effects
@@
 			)
 		)
-		(property "JLCPCB Rotation Offset" "0"
+		(property "JLCPCB Rotation Offset" ""
 			(at 41.91 30.48 0)
 			(effects
@@
 			)
 		)
-		(property "JLCPCB Rotation Offset" "0"
+		(property "JLCPCB Rotation Offset" ""
 			(at 259.08 218.44 0)
 			(effects
@@
 			)
 		)
-		(property "JLCPCB Rotation Offset" "0"
+		(property "JLCPCB Rotation Offset" ""
 			(at 38.1 102.87 0)
 			(effects
@@
 			)
 		)
-		(property "JLCPCB Rotation Offset" "0"
+		(property "JLCPCB Rotation Offset" ""
 			(at 261.62 251.46 0)
 			(effects

Commit message: Update jlc part num for CH340 Fixes#346
Parts:
- U7: JLCPCB Part # C84681 -> C7464026
Changed lines of the file:
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@@
 			)
 		)
-		(property "JLCPCB Part #" "C84681"
+		(property "JLCPCB Part #" "C7464026"
 			(at 330.2 189.23 0)
 			(effects

Commit message: update all harware revs
Parts:
- Y1: value 16MHz -> 16MHz
- gave numbers to parts that had none: 29
Other:
- moved on the sheet: JP6
