File: hardware/disp_A/disp_A.kicad_sch (KiCad schematic)
At the start: 115 parts, among them J1 Conn_02x16_Odd_Even_FLIP, J2 Conn_01x01_Pin, J3 Conn_01x01_Pin, Q1 2N7002, Q10 2N7002, Q11 2N7002, Q12 2N7002, Q13 2N7002, Q2 2N7002, Q3 2N7002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

Commit message: fix rotation on disp
Parts:
- Q1, Q10, Q11, Q12, Q13, Q2, Q3, Q4, Q5, Q6, Q7, Q8, Q9: JLCPCB Rotation Offset 180 -> (none)
Changed lines of the file:
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@@
 			)
 		)
-		(property "JLCPCB Rotation Offset" "180"
+		(property "JLCPCB Rotation Offset" ""
 			(at 27.94 190.5 0)
 			(effects
@@
 			)
 		)
-		(property "JLCPCB Rotation Offset" "180"
+		(property "JLCPCB Rotation Offset" ""
 			(at 114.3 189.23 0)
 			(effects
@@
 			)
 		)
-		(property "JLCPCB Rotation Offset" "180"
+		(property "JLCPCB Rotation Offset" ""
 			(at 144.78 189.23 0)
 			(effects
@@
 			)
 		)
-		(property "JLCPCB Rotation Offset" "180"
+		(property "JLCPCB Rotation Offset" ""
 			(at 111.76 52.07 0)
 			(effects
@@
 			)
 		)
-		(property "JLCPCB Rotation Offset" "180"
+		(property "JLCPCB Rotation Offset" ""
 			(at 111.76 72.39 0)
 			(effects
@@
 			)
 		)
-		(property "JLCPCB Rotation Offset" "180"
+		(property "JLCPCB Rotation Offset" ""
 			(at 29.21 140.97 0)
 			(effects
@@
 			)
 		)
-		(property "JLCPCB Rotation Offset" "180"
+		(property "JLCPCB Rotation Offset" ""
 			(at 59.69 140.97 0)
 			(effects
@@
 			)
 		)
-		(property "JLCPCB Rotation Offset" "180"
+		(property "JLCPCB Rotation Offset" ""
 			(at 115.57 142.24 0)
 			(effects
@@
 			)
 		)
-		(property "JLCPCB Rotation Offset" "180"
+		(property "JLCPCB Rotation Offset" ""
 			(at 85.09 189.23 0)
 			(effects
@@
 			)
 		)
-		(property "JLCPCB Rotation Offset" "180"
+		(property "JLCPCB Rotation Offset" ""
 			(at 144.78 140.97 0)
 			(effects
@@
 			)
 		)
-		(property "JLCPCB Rotation Offset" "180"
+		(property "JLCPCB Rotation Offset" ""
 			(at 110.49 33.02 0)
 			(effects
@@
 			)
 		)
-		(property "JLCPCB Rotation Offset" "180"
+		(property "JLCPCB Rotation Offset" ""
 			(at 86.36 140.97 0)
 			(effects
@@
 			)
 		)
-		(property "JLCPCB Rotation Offset" "180"
+		(property "JLCPCB Rotation Offset" ""
 			(at 59.69 189.23 0)
 			(effects
